Commit message: Update Simulation Package

File: install/charmie_bot/share/charmie_bot/description/depth_camera.xacro (robot description, xacro)
@@ -1 +1,84 @@
-/home/utilizador/charmie_ws/src/charmie_bot/description/depth_camera.xacro
+<?xml version="1.0"?>
+<robot xmlns:xacro="http://www.ros.org/wiki/xacro">
+    <joint name="neck_joint" type="fixed">
+        <parent link="upper_body_link"/>
+        <child link="neck_link"/>
+        <origin xyz="0.045 0 0.5" rpy="0 0 0"/>
+    </joint>
+    <link name="neck_link">
+        <xacro:inertial_box mass="0.1" x="0" y="0" z="0">
+            <origin xyz="0 0 0" rpy="0 0 0"/>
+        </xacro:inertial_box>
+    </link>
+    <joint name="camera_joint_z" type="revolute">
+        <parent link="neck_link"/>
+        <child link="camera_link_z"/>
+        <origin xyz="0 0 0" rpy="0 0 0"/>
+        <axis xyz="0 1 0"/>
+        <limit effort="1000.0" lower="0.0" upper="0.548" velocity="0.5"/>
+    </joint>
+    <link name="camera_link_z">
+        <xacro:inertial_box mass="0.1" x="0" y="0" z="0">
+            <origin xyz="0 0 0" rpy="0 0 0"/>
+        </xacro:inertial_box>
+    </link>
+    <joint name="camera_joint_y" type="revolute">
+        <parent link="camera_link_z"/>
+        <child link="camera_link_y"/>
+        <origin xyz="0 0 0" rpy="0 0 0"/>
+        <axis xyz="0 0 1"/>
+        <limit effort="1000.0" lower="-0.548" upper="0.548" velocity="0.5"/>
+    </joint>
+    <link name="camera_link_y">
+        <xacro:inertial_box mass="0.1" x="0" y="0" z="0">
+            <origin xyz="0 0 0" rpy="0 0 0"/>
+        </xacro:inertial_box>
+    </link>
+    <joint name="camera_joint" type="fixed">
+        <parent link="camera_link_y"/>
+        <child link="camera_link"/>
+        <origin xyz="0 0 0" rpy="0 0 0"/>
+    </joint>
+    <link name="camera_link">
+        <visual>
+            <geometry>
+                <box size="0.04 0.07 0.04"/>
+            </geometry>
+            <material name="red"/>
+        </visual>
+        <xacro:inertial_box mass="0.1" x="0.04" y="0.07" z="0.04">
+            <origin xyz="0 0 0" rpy="0 0 0"/>
+        </xacro:inertial_box>
+    </link>
+    <joint name="camera_optical_joint" type="fixed">
+        <parent link="camera_link"/>
+        <child link="camera_link_optical"/>
+        <origin xyz="0 0 0" rpy="${-pi/2} 0 ${-pi/2}"/>
+    </joint>
+    <link name="camera_link_optical"></link>
+    <gazebo reference="camera_link">
+        <material>Gazebo/Red</material>
+        <sensor name="camera" type="depth">
+            <pose> 0 0 0 0 0 0 </pose>
+            <visualize>true</visualize>
+            <update_rate>10</update_rate>
+            <camera>
+                <horizontal_fov>1.089</horizontal_fov>
+                <image>
+                    <format>B8G8R8</format>
+                    <width>640</width>
+                    <height>480</height>
+                </image>
+                <clip>
+                    <near>0.05</near>
+                    <far>8.0</far>
+                </clip>
+            </camera>
+            <plugin name="camera_controller" filename="libgazebo_ros_camera.so">
+                <frame_name>camera_link_optical</frame_name>
+                <min_depth>0.1</min_depth>
+                <max_depth>100.0</max_depth>
+            </plugin>
+        </sensor>
+    </gazebo>
+</robot>

File: install/charmie_bot/share/charmie_bot/description/gazebo_control.xacro (robot description, xacro)
@@ -1 +1,19 @@
-/home/utilizador/charmie_ws/src/charmie_bot/description/gazebo_control.xacro
+<?xml version="1.0"?>
+<robot xmlns:xacro="http://www.ros.org/wiki/xacro">
+    <gazebo>
+        <plugin name="omni_steering" filename="libgazebo_ros_planar_move.so">
+            <commandTopic>cmd_vel</commandTopic>
+            <odometry_rate>100.0</odometry_rate>
+            <odometry_frame>odom</odometry_frame>
+            <robot_base_frame>base_link</robot_base_frame>
+            <publish_odom>true</publish_odom>
+            <publish_odom_tf>true</publish_odom_tf>
+            <publish_wheel_tf>true</publish_wheel_tf>
+        </plugin>
+    </gazebo>
+    <gazebo>
+        <plugin name="gazebo_ros_control" filename="libgazebo_ros_control.so">
+            <robotNamespace>robot</robotNamespace>
+        </plugin>
+    </gazebo>
+</robot>

File: install/charmie_bot/share/charmie_bot/description/lidar.xacro (robot description, xacro)
@@ -1 +1,55 @@
-/home/utilizador/charmie_ws/src/charmie_bot/description/lidar.xacro
+<?xml version="1.0"?>
+<robot xmlns:xacro="http://www.ros.org/wiki/xacro" >
+    <joint name="laser_joint" type="fixed">
+        <parent link="chassi_link"/>
+        <child link="lidar_frame"/>
+        <origin xyz="0 0.2 0.177" rpy="0 0 ${pi/2}"/>
+    </joint>
+    <link name="lidar_frame">
+        <visual>
+            <origin xyz="0 0 -0.055" rpy="${pi/2} 0 ${pi}"/>
+            <geometry>
+                <mesh filename="file://$(find charmie_bot)/description/meshes/lidar.stl" scale="0.001 0.001 0.001"/>
+                <!-- <cylinder radius="0.05" length="0.04"/> -->
+            </geometry>
+            <material name="red"/>
+        </visual>
+        <collision>
+            <geometry>
+                <cylinder radius="0.05" length="0.04"/>
+            </geometry>
+        </collision>
+        <xacro:inertial_cylinder mass="0.1" length="0.04" radius="0.05">
+            <origin xyz="0 0 0" rpy="0 0 0"/>
+        </xacro:inertial_cylinder>
+    </link>
+    <!-- hokuyo -->
+    <gazebo reference="lidar_frame">
+        <material>Gazebo/Red</material>
+        <sensor type="ray" name="head_hokuyo_sensor">
+            <pose> 0 0 0.055 0 0 0 </pose>
+            <visualize>true</visualize>
+            <update_rate>40</update_rate>
+            <ray>
+                <scan>
+                    <horizontal>
+                        <samples>681</samples>
+                        <min_angle>-2.092387973753402</min_angle>
+                        <max_angle>2.092387973753402</max_angle>
+                    </horizontal>
+                </scan>
+                <range>
+                    <min>0.2</min>
+                    <max>5.6</max>
+                </range>
+            </ray>
+            <plugin name="laser_controller" filename="libgazebo_ros_ray_sensor.so">
+                <ros>
+                    <argument>~/out:=scan</argument>
+                </ros>
+                <output_type>sensor_msgs/LaserScan</output_type>
+                <frame_name>lidar_frame</frame_name>
+            </plugin>
+        </sensor>
+    </gazebo>
+</robot>

File: install/charmie_bot/share/charmie_bot/description/robot.urdf.xacro (robot description, xacro)
@@ -1 +1,7 @@
-/home/utilizador/charmie_ws/src/charmie_bot/description/robot.urdf.xacro
+<?xml version="1.0"?>
+<robot xmlns:xacro="http://www.ros.org/wiki/xacro"  name="robot">
+    <xacro:include filename='robot_core.xacro'/>
+    <xacro:include filename='robot_wheels.xacro'/>
+    <xacro:include filename='lidar.xacro'/>
+    <xacro:include filename='gazebo_control.xacro'/>
+</robot>

File: install/charmie_bot/share/charmie_bot/description/robot_core.xacro (robot description, xacro)
@@ -1 +1,117 @@
-/home/utilizador/charmie_ws/src/charmie_bot/description/robot_core.xacro
+<?xml version="1.0"?>
+<robot xmlns:xacro="http://www.ros.org/wiki/xacro" >
+    <xacro:include filename="inertial_macros.xacro"/>
+    <material name="white">
+        <color rgba="1 1 1 1"/>
+    </material>
+    <material name="blue">
+        <color rgba="0.2 0.2 1 1"/>
+    </material>
+    <material name="black">
+        <color rgba="0 0 0 1"/>
+    </material>
+    <material name="red">
+        <color rgba="1 0 0 1"/>
+    </material>
+    <material name="grey">
+        <color rgba="0.5 0.5 0.5 1"/>
+    </material>
+    <!--BASE LINK-->
+    <link name="base_link">
+    </link>
+    <!--BASE FOOTPRINT-->
+    <joint name="base_footprint_joint" type="fixed">
+        <parent link="base_link"/>
+        <child link="base_footprint"/>
+        <origin xyz="0 0 0" rpy="0 0 0"/>
+    </joint>
+    <link name="base_footprint">
+    </link>
+    <!--CHASSI-->
+    <joint name="chassi_joint" type="fixed">
+        <parent link="base_link"/>
+        <child link="chassi_link"/>
+        <!-- <origin xyz="0 0 0.085"/> -->
+        <origin xyz="0 0 0.082" rpy="0 0 0"/>
+    </joint>
+    <link name="chassi_link">
+        <visual>
+            <origin xyz="0 0 0"/>
+            <geometry>
+                <cylinder radius="0.275" length="0.25"/>
+            </geometry>
+            <material name="white"/>
+        </visual>
+        <collision>
+            <origin xyz="0 0 0"/>
+            <geometry>
+                <cylinder radius="0.275" length="0.25"/>
+            </geometry>
+        </collision>
+        <xacro:inertial_cylinder mass="1.0" length="0.25" radius="0.275">
+            <origin xyz="0 0 0" rpy="0 0 0"/>
+        </xacro:inertial_cylinder>
+    </link>
+    <gazebo reference="chassi_link">
+        <material>Gazebo/White</material>
+    </gazebo>
+    <!--LOWER BODY-->
+    <joint name="lower_body_joint" type="fixed">
+        <parent link="base_link"/>
+        <child link="lower_body_link"/>
+        <origin xyz="0 0 0.2" rpy="0 0 ${pi/2}"/>
+        <!-- <axis xyz="0 0 1"/>
+        <limit lower="0" upper="0.14" velocity="100" effort="100"/> -->
+    </joint>
+    <link name="lower_body_link">
+        <visual>
+            <origin xyz="0 0 0.18" rpy="0 0 ${pi/2}"/>
+            <geometry>
+                <box size="0.2 0.05 0.35"/>
+            </geometry>
+            <material name="white"/>
+        </visual>
+        <collision>
+            <origin xyz="0 0 0.18" rpy="0 0 ${pi/2}"/>
+            <geometry>
+                <box size="0.2 0.05 0.35"/>
+            </geometry>
+        </collision>
+        <xacro:inertial_box mass="0.1" x="0.2" y="0.05" z="0.35">
+            <origin xyz="0 0 0.18" rpy="0 0 0"/>
+        </xacro:inertial_box>
+    </link>
+    <gazebo reference="lower_body_link">
+        <material>Gazebo/White</material>
+    </gazebo>
+    <!--UPPER BODY-->
+    <joint name="upper_body_joint" type="fixed">
+        <parent link="lower_body_link"/>
+        <child link="upper_body_link"/>
+        <origin xyz="0 0 0.355" rpy="0 0 0"/>
+        <!-- <axis xyz="0 1 0"/>
+        <limit lower="0.1745" upper="1.2217" velocity="100" effort="100"/> -->
+    </joint>
+    <link name="upper_body_link">
+        <visual>
+            <origin xyz="0 0 0.25" rpy="0 0 ${pi/2}"/>
+            <geometry>
+                <box size="0.2 0.05 0.50"/>
+            </geometry>
+            <material name="white"/>
+        </visual>
+        <collision>
+            <origin xyz="0 0 0.25" rpy="0 0 ${pi/2}"/>
+            <geometry>
+                <box size="0.2 0.05 0.50"/>
+            </geometry>
+        </collision>
+        <xacro:inertial_box mass="0.03" x="0.2" y="0.05" z="0.50">
+            <origin xyz="0 0 0.25" rpy="0 0 0"/>
+        </xacro:inertial_box>
+    </link>
+    <gazebo reference="upper_body_link">
+        <material>Gazebo/White</material>
+    </gazebo>
+    <!-- <xacro: omni_steering/>  -->
+</robot>

File: install/charmie_bot/share/charmie_bot/description/robot_wheels.xacro (robot description, xacro)
@@ -1 +1,116 @@
-/home/utilizador/charmie_ws/src/charmie_bot/description/robot_wheels.xacro
+<?xml version="1.0"?>
+<robot xmlns:xacro="http://www.ros.org/wiki/xacro">
+    <!--WHEELS-->
+    <!--LEFT FRONT-->
+    <joint name="left_front_joint" type="fixed">
+        <parent link="base_link"/>
+        <child link="left_front_link"/>
+        <origin xyz="0.2 0.2 0" rpy="-${pi/2} 0 -${pi/4}"/>
+    </joint>
+    <link name="left_front_link">
+        <visual>
+            <geometry>
+                <mesh filename="file://$(find charmie_bot)/description/meshes/omni_wheel.stl" scale="0.001 0.001 0.001"/>
+                <!-- <cylinder radius="0.105" length="0.04"/> -->
+            </geometry>
+            <material name="grey"/>
+        </visual>
+        <collision>
+            <geometry>
+                <cylinder radius="0.105" length="0.04"/>
+            </geometry>
+        </collision>
+        <xacro:inertial_cylinder mass="0.1" length="0.04" radius="0.105">
+            <origin xyz="0 0 0" rpy="0 0 0"/>
+        </xacro:inertial_cylinder>
+    </link>
+    <gazebo reference="left_front_link">
+        <material>Gazebo/Grey</material>
+        <mu1 value="0.001"/>
+        <mu2 value="0.001"/>
+    </gazebo>
+    <!--LEFT BACK-->
+    <joint name="left_back_joint" type="fixed">
+        <parent link="base_link"/>
+        <child link="left_back_link"/>
+        <origin xyz="-0.2 0.2 0" rpy="0 -${pi/2} -${pi/4}"/>
+    </joint>
+    <link name="left_back_link">
+        <visual>
+            <geometry>
+                <mesh filename="file://$(find charmie_bot)/description/meshes/omni_wheel.stl" scale="0.001 0.001 0.001"/>
+                <!--<cylinder radius="0.1" length="0.04"/>-->
+            </geometry>
+            <material name="grey"/>
+        </visual>
+        <collision>
+            <geometry>
+                <cylinder radius="0.105" length="0.04"/>
+            </geometry>
+        </collision>
+        <xacro:inertial_cylinder mass="0.1" length="0.04" radius="0.105">
+            <origin xyz="0 0 0" rpy="0 0 0"/>
+        </xacro:inertial_cylinder>
+    </link>
+    <gazebo reference="left_back_link">
+        <material>Gazebo/Grey</material>
+        <mu1 value="0.001"/>
+        <mu2 value="0.001"/>
+    </gazebo>
+    <!--RIGHT FRONT-->
+    <joint name="right_front_joint" type="fixed">
+        <parent link="base_link"/>
+        <child link="right_front_link"/>
+        <origin xyz="0.2 -0.2 0" rpy="0 ${pi/2} -${pi/4}"/>
+    </joint>
+    <link name="right_front_link">
+        <visual>
+            <geometry>
+                <mesh filename="file://$(find charmie_bot)/description/meshes/omni_wheel.stl" scale="0.001 0.001 0.001"/>
+                <!--<cylinder radius="0.1" length="0.04"/>-->
+            </geometry>
+            <material name="grey"/>
+        </visual>
+        <collision>
+            <geometry>
+                <cylinder radius="0.105" length="0.04"/>
+            </geometry>
+        </collision>
+        <xacro:inertial_cylinder mass="0.1" length="0.04" radius="0.105">
+            <origin xyz="0 0 0" rpy="0 0 0"/>
+        </xacro:inertial_cylinder>
+    </link>
+    <gazebo reference="right_front_link">
+        <material>Gazebo/Grey</material>
+        <mu1 value="0.001"/>
+        <mu2 value="0.001"/>
+    </gazebo>
+    <!--RIGHT BACK-->
+    <joint name="right_back_joint" type="fixed">
+        <parent link="base_link"/>
+        <child link="right_back_link"/>
+        <origin xyz="-0.2 -0.2 0" rpy="${pi/2} 0 -${pi/4}"/>
+    </joint>
+    <link name="right_back_link">
+        <visual>
+            <geometry>
+                <mesh filename="file://$(find charmie_bot)/description/meshes/omni_wheel.stl" scale="0.001 0.001 0.001"/>
+                <!--<cylinder radius="0.1" length="0.04"/>-->
+            </geometry>
+            <material name="grey"/>
+        </visual>
+        <collision>
+            <geometry>
+                <cylinder radius="0.105" length="0.04"/>
+            </geometry>
+        </collision>
+        <xacro:inertial_cylinder mass="0.1" length="0.04" radius="0.105">
+            <origin xyz="0 0 0" rpy="0 0 0"/>
+        </xacro:inertial_cylinder>
+    </link>
+    <gazebo reference="right_back_link">
+        <material>Gazebo/Grey</material>
+        <mu1 value="0.001"/>
+        <mu2 value="0.001"/>
+    </gazebo>
+</robot>

File: src/charmie_bot/description/lidar.xacro (robot description, xacro)
@@ -3,8 +3,8 @@
     <joint name="laser_joint" type="fixed">
         <parent link="chassi_link"/>
-        <child link="laser_frame"/>
+        <child link="lidar_frame"/>
         <origin xyz="0 0.2 0.177" rpy="0 0 ${pi/2}"/>
     </joint>
-    <link name="laser_frame">
+    <link name="lidar_frame">
         <visual>
             <origin xyz="0 0 -0.055" rpy="${pi/2} 0 ${pi}"/>
@@ -24,10 +24,11 @@
         </xacro:inertial_cylinder>
     </link>
-    <gazebo reference="laser_frame">
+    <!-- hokuyo -->
+    <gazebo reference="lidar_frame">
         <material>Gazebo/Red</material>
-        <sensor name="laser" type="ray">
+        <sensor type="ray" name="head_hokuyo_sensor">
             <pose> 0 0 0.055 0 0 0 </pose>
             <visualize>true</visualize>
-            <update_rate>10</update_rate>
+            <update_rate>40</update_rate>
             <ray>
                 <scan>
@@ -48,5 +49,5 @@
                 </ros>
                 <output_type>sensor_msgs/LaserScan</output_type>
-                <frame_name>laser_frame</frame_name>
+                <frame_name>lidar_frame</frame_name>
             </plugin>
         </sensor>

File: src/charmie_bot/description/robot.urdf.xacro (robot description, xacro)
@@ -4,5 +4,4 @@
     <xacro:include filename='robot_wheels.xacro'/>
     <xacro:include filename='lidar.xacro'/>
-    <!-- <xacro:include filename='depth_camera.xacro'/> -->
     <xacro:include filename='gazebo_control.xacro'/>
 </robot>
