Commit message: Last tweaks to localisation

File: src/charmie_bot/description/lidar.xacro (robot description, xacro)
@@ -4,5 +4,5 @@
         <parent link="chassi_link"/>
         <child link="lidar_frame"/>
-        <origin xyz="0 0.2 0.177" rpy="0 0 ${pi/2}"/>
+        <origin xyz="0.2 0 0.177" rpy="0 0 0"/>
     </joint>
     <link name="lidar_frame">
