Commit message: Added Newer Simulation Version and adjusted Odometry Publishing

File: src/charmie_bot/description/depth_camera.xacro (robot description, xacro)
@@ -4,5 +4,5 @@
         <parent link="upper_body_link"/>
         <child link="neck_link"/>
-        <origin xyz="0.045 0 0.8" rpy="0 0 0"/>
+        <origin xyz="0.045 0 0.5" rpy="0 0 0"/>
     </joint>
     <link name="neck_link">
@@ -66,5 +66,5 @@
                 <horizontal_fov>1.089</horizontal_fov>
                 <image>
-                    <format>R8G8B8</format>
+                    <format>B8G8R8</format>
                     <width>640</width>
                     <height>480</height>
@@ -77,4 +77,6 @@
             <plugin name="camera_controller" filename="libgazebo_ros_camera.so">
                 <frame_name>camera_link_optical</frame_name>
+                <min_depth>0.1</min_depth>
+                <max_depth>100.0</max_depth>
             </plugin>
         </sensor>

File: src/charmie_bot/description/gazebo_control.xacro (robot description, xacro)
@@ -1,21 +1,19 @@
 <?xml version="1.0"?>
 <robot xmlns:xacro="http://www.ros.org/wiki/xacro">
-    <xacro:macro name="omni_steering" params="">
-        <gazebo>
-            <plugin name="omni_steering" filename="libgazebo_ros_planar_move.so">
-                <commandTopic>cmd_vel</commandTopic>
-                <odometry_rate>100.0</odometry_rate>
-                <odometry_frame>odom</odometry_frame>
-                <robot_base_frame>base_link</robot_base_frame>
-                <publish_odom>true</publish_odom>
-                <publish_odom_tf>true</publish_odom_tf>
-                <publish_wheel_tf>true</publish_wheel_tf>
-            </plugin>
-        </gazebo>
-    </xacro:macro>
-    <!-- <gazebo>
+    <gazebo>
+        <plugin name="omni_steering" filename="libgazebo_ros_planar_move.so">
+            <commandTopic>cmd_vel</commandTopic>
+            <odometry_rate>100.0</odometry_rate>
+            <odometry_frame>odom</odometry_frame>
+            <robot_base_frame>base_link</robot_base_frame>
+            <publish_odom>true</publish_odom>
+            <publish_odom_tf>true</publish_odom_tf>
+            <publish_wheel_tf>true</publish_wheel_tf>
+        </plugin>
+    </gazebo>
+    <gazebo>
         <plugin name="gazebo_ros_control" filename="libgazebo_ros_control.so">
             <robotNamespace>robot</robotNamespace>
         </plugin>
-    </gazebo> -->
+    </gazebo>
 </robot>

File: src/charmie_bot/description/lidar.xacro (robot description, xacro)
@@ -1,13 +1,15 @@
 <?xml version="1.0"?>
-<robot xmlns:xacro="http://www.ros.org/wiki/xacro">
-    <joint name="lidar_joint" type="fixed">
+<robot xmlns:xacro="http://www.ros.org/wiki/xacro" >
+    <joint name="laser_joint" type="fixed">
         <parent link="chassi_link"/>
-        <child link="lidar_frame"/>
-        <origin xyz="0.2 0 0.18" rpy="0 0 0"/>
+        <child link="laser_frame"/>
+        <origin xyz="0 0.2 0.177" rpy="0 0 ${pi/2}"/>
     </joint>
-    <link name="lidar_frame">
+    <link name="laser_frame">
         <visual>
+            <origin xyz="0 0 -0.055" rpy="${pi/2} 0 ${pi}"/>
             <geometry>
-                <cylinder radius="0.05" length="0.04"/>
+                <mesh filename="file://$(find charmie_bot)/description/meshes/lidar.stl" scale="0.001 0.001 0.001"/>
+                <!-- <cylinder radius="0.05" length="0.04"/> -->
             </geometry>
             <material name="red"/>
@@ -22,8 +24,8 @@
         </xacro:inertial_cylinder>
     </link>
-    <gazebo reference="lidar_frame">
+    <gazebo reference="laser_frame">
         <material>Gazebo/Red</material>
         <sensor name="laser" type="ray">
-            <pose> 0 0 0 0 0 0 </pose>
+            <pose> 0 0 0.055 0 0 0 </pose>
             <visualize>true</visualize>
             <update_rate>10</update_rate>
@@ -31,12 +33,12 @@
                 <scan>
                     <horizontal>
-                        <samples>360</samples>
-                        <min_angle>-2.356</min_angle> <!--180 degrees-->
-                        <max_angle>2.356</max_angle>
+                        <samples>681</samples>
+                        <min_angle>-2.092387973753402</min_angle>
+                        <max_angle>2.092387973753402</max_angle>
                     </horizontal>
                 </scan>
                 <range>
-                    <min>0.3</min>
-                    <max>12</max>
+                    <min>0.2</min>
+                    <max>5.6</max>
                 </range>
             </ray>
@@ -46,5 +48,5 @@
                 </ros>
                 <output_type>sensor_msgs/LaserScan</output_type>
-                <frame_name>lidar_frame</frame_name>
+                <frame_name>laser_frame</frame_name>
             </plugin>
         </sensor>

File: src/charmie_bot/description/robot.urdf.xacro (robot description, xacro)
@@ -1,8 +1,8 @@
 <?xml version="1.0"?>
 <robot xmlns:xacro="http://www.ros.org/wiki/xacro"  name="robot">
-    <xacro:include filename="robot_core_Rui.xacro" />
-    <xacro:include filename="lidar.xacro" />
-    <xacro:include filename="camera.xacro" />
-    <!--<xacro:include filename="left_arm.xacro" />
-    <xacro:include filename="right_arm.xacro" />-->
+    <xacro:include filename='robot_core.xacro'/>
+    <xacro:include filename='robot_wheels.xacro'/>
+    <xacro:include filename='lidar.xacro'/>
+    <!-- <xacro:include filename='depth_camera.xacro'/> -->
+    <xacro:include filename='gazebo_control.xacro'/>
 </robot>

File: src/charmie_bot/description/robot_core.xacro (robot description, xacro)
@@ -2,5 +2,4 @@
 <robot xmlns:xacro="http://www.ros.org/wiki/xacro" >
     <xacro:include filename="inertial_macros.xacro"/>
-    <xacro:include filename="gazebo_control.xacro" />
     <material name="white">
         <color rgba="1 1 1 1"/>
@@ -15,113 +14,104 @@
         <color rgba="1 0 0 1"/>
     </material>
-    <!-- BASE LINK -->
+    <material name="grey">
+        <color rgba="0.5 0.5 0.5 1"/>
+    </material>
+    <!--BASE LINK-->
     <link name="base_link">
     </link>
-    <!-- CHASSIS LINK -->
-    <joint name="chassis_joint" type="fixed">
+    <!--BASE FOOTPRINT-->
+    <joint name="base_footprint_joint" type="fixed">
         <parent link="base_link"/>
-        <child link="chassis"/>
-        <origin xyz="-0.1 0 0"/>
+        <child link="base_footprint"/>
+        <origin xyz="0 0 0" rpy="0 0 0"/>
     </joint>
-    <link name="chassis">
+    <link name="base_footprint">
+    </link>
+    <!--CHASSI-->
+    <joint name="chassi_joint" type="fixed">
+        <parent link="base_link"/>
+        <child link="chassi_link"/>
+        <!-- <origin xyz="0 0 0.085"/> -->
+        <origin xyz="0 0 0.082" rpy="0 0 0"/>
+    </joint>
+    <link name="chassi_link">
         <visual>
-            <origin xyz="0.15 0 0.075"/>
+            <origin xyz="0 0 0"/>
             <geometry>
-                <box size="0.3 0.3 0.15"/>
+                <cylinder radius="0.275" length="0.25"/>
             </geometry>
             <material name="white"/>
         </visual>
         <collision>
-            <origin xyz="0.15 0 0.075"/>
+            <origin xyz="0 0 0"/>
             <geometry>
-                <box size="0.3 0.3 0.15"/>
+                <cylinder radius="0.275" length="0.25"/>
             </geometry>
         </collision>
-        <xacro:inertial_box mass="0.5" x="0.3" y="0.3" z="0.15">
-            <origin xyz="0.15 0 0.075" rpy="0 0 0"/>
-        </xacro:inertial_box>
-    </link>
-    <gazebo reference="chassis">
-        <material>Gazebo/White</material>
-    </gazebo>
-    <!-- LEFT WHEEL LINK -->
-    <joint name="left_wheel_joint" type="continuous">
-        <parent link="base_link"/>
-        <child link="left_wheel"/>
-        <origin xyz="0 0.175 0" rpy="-${pi/2} 0 0" />
-        <axis xyz="0 0 1"/>
-    </joint>
-    <link name="left_wheel">
-        <visual>
-            <geometry>
-                <cylinder radius="0.05" length="0.04"/>
-            </geometry>
-            <material name="blue"/>
-        </visual>
-        <collision>
-            <geometry>
-                <cylinder radius="0.05" length="0.04"/>
-            </geometry>
-        </collision>
-        <xacro:inertial_cylinder mass="0.1" length="0.04" radius="0.05">
+        <xacro:inertial_cylinder mass="1.0" length="0.25" radius="0.275">
             <origin xyz="0 0 0" rpy="0 0 0"/>
         </xacro:inertial_cylinder>
     </link>
-    <gazebo reference="left_wheel">
-        <material>Gazebo/Blue</material>
+    <gazebo reference="chassi_link">
+        <material>Gazebo/White</material>
     </gazebo>
-    <!-- RIGHT WHEEL LINK -->
-    <joint name="right_wheel_joint" type="continuous">
+    <!--LOWER BODY-->
+    <joint name="lower_body_joint" type="fixed">
         <parent link="base_link"/>
-        <child link="right_wheel"/>
-        <origin xyz="0 -0.175 0" rpy="${pi/2} 0 0" />
-        <axis xyz="0 0 -1"/>
+        <child link="lower_body_link"/>
+        <origin xyz="0 0 0.2" rpy="0 0 ${pi/2}"/>
+        <!-- <axis xyz="0 0 1"/>
+        <limit lower="0" upper="0.14" velocity="100" effort="100"/> -->
     </joint>
-    <link name="right_wheel">
+    <link name="lower_body_link">
         <visual>
+            <origin xyz="0 0 0.18" rpy="0 0 ${pi/2}"/>
             <geometry>
-                <cylinder radius="0.05" length="0.04"/>
+                <box size="0.2 0.05 0.35"/>
             </geometry>
-            <material name="blue"/>
+            <material name="white"/>
         </visual>
         <collision>
+            <origin xyz="0 0 0.18" rpy="0 0 ${pi/2}"/>
             <geometry>
-                <cylinder radius="0.05" length="0.04"/>
+                <box size="0.2 0.05 0.35"/>
             </geometry>
         </collision>
-        <xacro:inertial_cylinder mass="0.1" length="0.04" radius="0.05">
-            <origin xyz="0 0 0" rpy="0 0 0"/>
-        </xacro:inertial_cylinder>
+        <xacro:inertial_box mass="0.1" x="0.2" y="0.05" z="0.35">
+            <origin xyz="0 0 0.18" rpy="0 0 0"/>
+        </xacro:inertial_box>
     </link>
-    <gazebo reference="right_wheel">
-        <material>Gazebo/Blue</material>
+    <gazebo reference="lower_body_link">
+        <material>Gazebo/White</material>
     </gazebo>
-    <!-- CASTER WHEEL LINK -->
-    <joint name="caster_wheel_joint" type="fixed">
-        <parent link="chassis"/>
-        <child link="caster_wheel"/>
-        <origin xyz="0.24 0 0"/>
+    <!--UPPER BODY-->
+    <joint name="upper_body_joint" type="fixed">
+        <parent link="lower_body_link"/>
+        <child link="upper_body_link"/>
+        <origin xyz="0 0 0.355" rpy="0 0 0"/>
+        <!-- <axis xyz="0 1 0"/>
+        <limit lower="0.1745" upper="1.2217" velocity="100" effort="100"/> -->
     </joint>
-    <link name="caster_wheel">
+    <link name="upper_body_link">
         <visual>
+            <origin xyz="0 0 0.25" rpy="0 0 ${pi/2}"/>
             <geometry>
-                <sphere radius="0.05"/>
+                <box size="0.2 0.05 0.50"/>
             </geometry>
-            <material name="black"/>
+            <material name="white"/>
         </visual>
         <collision>
+            <origin xyz="0 0 0.25" rpy="0 0 ${pi/2}"/>
             <geometry>
-                <sphere radius="0.05"/>
+                <box size="0.2 0.05 0.50"/>
             </geometry>
         </collision>
-        <xacro:inertial_sphere mass="0.1" radius="0.05">
-            <origin xyz="0 0 0" rpy="0 0 0"/>
-        </xacro:inertial_sphere>
+        <xacro:inertial_box mass="0.03" x="0.2" y="0.05" z="0.50">
+            <origin xyz="0 0 0.25" rpy="0 0 0"/>
+        </xacro:inertial_box>
     </link>
-    <gazebo reference="caster_wheel">
-        <material>Gazebo/Black</material>
-        <mu1 value="0.001"/>
-        <mu2 value="0.001"/>
+    <gazebo reference="upper_body_link">
+        <material>Gazebo/White</material>
     </gazebo>
-    <xacro:omni_steering/>
+    <!-- <xacro: omni_steering/>  -->
 </robot>

Commit message: Added the new package compatible with version 22.04 of Ubuntu and Humble of ROS2. Tested in the camera RSd405. Also added the camera to URDF File

File: src/charmie_bot/description/depth_camera.xacro (robot description, xacro)
@@ -38,5 +38,5 @@
         <parent link="camera_link_y"/>
         <child link="camera_link"/>
-        <origin xyz="0 0 0" rpy="0 0 0"/>
+        <origin xyz="0 0 0.05" rpy="0 0 0"/>
     </joint>
     <link name="camera_link">
@@ -45,5 +45,5 @@
                 <box size="0.04 0.07 0.04"/>
             </geometry>
-            <material name="red"/>
+            <material name="blue"/>
         </visual>
         <xacro:inertial_box mass="0.1" x="0.04" y="0.07" z="0.04">
@@ -58,5 +58,5 @@
     <link name="camera_link_optical"></link>
     <gazebo reference="camera_link">
-        <material>Gazebo/Red</material>
+        <material>Gazebo/Blue</material>
         <sensor name="camera" type="depth">
             <pose> 0 0 0 0 0 0 </pose>

File: src/charmie_bot/description/robot.urdf.xacro (robot description, xacro)
@@ -4,4 +4,5 @@
     <xacro:include filename='robot_wheels.xacro'/>
     <xacro:include filename='lidar.xacro'/>
+    <xacro:include filename='depth_camera.xacro'/>
     <xacro:include filename='gazebo_control.xacro'/>
     <xacro:include filename='xarm6.urdf.xacro'/>
