Commit message: Updated the xarm_ros package to the one with moveit and with some parameteres redefined

File: src/charmie_arm_ufactory/xarm_ros2/xarm_description/urdf/camera/realsense_d435i.urdf.xacro (robot description, xacro)
@@ -16,9 +16,14 @@
     </link>
     <xacro:if value="${add_d435i_links}">
-      <link name="${prefix}camera_link"></link>
+      <!-- <link name="${prefix}camera_link"></link>
       <link name="${prefix}camera_depth_frame"></link>
       <link name="${prefix}camera_depth_optical_frame"></link>
       <link name="${prefix}camera_color_frame"></link>
-      <link name="${prefix}camera_color_optical_frame"></link>
+      <link name="${prefix}camera_color_optical_frame"></link> -->
+      <link name="${prefix}D405_hand_link"></link>
+      <link name="${prefix}D405_hand_depth_frame"></link>
+      <link name="${prefix}D405_hand_depth_optical_frame"></link>
+      <link name="${prefix}D405_hand_color_frame"></link>
+      <link name="${prefix}D405_hand_color_optical_frame"></link>
       <link name="${prefix}camera_left_ir_frame"></link>
       <link name="${prefix}camera_left_ir_optical_frame"></link>
@@ -27,29 +32,29 @@
       <joint name="${prefix}camera_link_joint" type="fixed">
         <parent link="${prefix}link_eef" />
-        <child link="${prefix}camera_link" />
+        <child link="${prefix}D405_hand_link" />
         <origin xyz="0.06746 -0.0175 0.0237" rpy="${M_PI} ${-M_PI/2} 0" />
       </joint>
       <joint name="${prefix}camera_depth_joint" type="fixed">
-        <parent link="${prefix}camera_link" />
-        <child link="${prefix}camera_depth_frame" />
+        <parent link="${prefix}D405_hand_link" />
+        <child link="${prefix}D405_hand_depth_frame" />
         <origin xyz="0 0 0" rpy="0 0 0" />
       </joint>
       <joint name="${prefix}camera_depth_optical_joint" type="fixed">
-        <parent link="${prefix}camera_depth_frame" />
-        <child link="${prefix}camera_depth_optical_frame" />
+        <parent link="${prefix}D405_hand_depth_frame" />
+        <child link="${prefix}D405_hand_depth_optical_frame" />
         <origin xyz="0 0 0" rpy="${-M_PI/2} 0 ${-M_PI/2}" />
       </joint>
       <joint name="${prefix}camera_color_joint" type="fixed">
-        <parent link="${prefix}camera_link" />
-        <child link="${prefix}camera_color_frame" />
+        <parent link="${prefix}D405_hand_link" />
+        <child link="${prefix}D405_hand_color_frame" />
         <origin xyz="0 0.015 0" rpy="0 0 0" />
       </joint>
       <joint name="${prefix}camera_color_optical_joint" type="fixed">
-        <parent link="${prefix}camera_color_frame" />
-        <child link="${prefix}camera_color_optical_frame" />
+        <parent link="${prefix}D405_hand_color_frame" />
+        <child link="${prefix}D405_hand_color_optical_frame" />
         <origin xyz="0 0 0" rpy="${-M_PI/2} 0 ${-M_PI/2}" />
       </joint>
       <joint name="${prefix}camera_left_ir_joint" type="fixed">
-        <parent link="${prefix}camera_link" />
+        <parent link="${prefix}D405_hand_link" />
         <child link="${prefix}camera_left_ir_frame" />
         <origin xyz="0 0 0" rpy="0 0 0" />
@@ -61,5 +66,5 @@
       </joint>
       <joint name="${prefix}camera_right_ir_joint" type="fixed">
-        <parent link="${prefix}camera_link" />
+        <parent link="${prefix}D405_hand_link" />
         <child link="${prefix}camera_right_ir_frame" />
         <origin xyz="0 -0.050 0" rpy="0 0 0" />

File: src/charmie_arm_ufactory/xarm_ros2/xarm_description/urdf/common/common.link.xacro (robot description, xacro)
@@ -63,4 +63,7 @@
       <xacro:property name="inertial_params_filename" value="xarm6_type12_HT_LDBR2"/>
     </xacro:if>
+    <xacro:if value="${dof == 7 and robot_type == 'xarm7_mirror'}">
+      <xacro:property name="inertial_params_filename" value="xarm7_type13_HT_BR2"/>
+    </xacro:if>
     <xacro:if value="${use_len}">
       <xacro:property name="robot_sn_len" value="${len(robot_sn)}" />

File: src/charmie_arm_ufactory/xarm_ros2/xarm_description/urdf/uf850/uf850_robot_macro.xacro (robot description, xacro)
@@ -7,4 +7,5 @@
     velocity_control:=false
     add_gripper:=false
+    add_bio_gripper:=false
     ros2_control_plugin:='uf_robot_hardware/UFRobotSystemHardware'
     robot_ip:=''
@@ -29,5 +30,5 @@
           velocity_control="${velocity_control}"
           ros2_control_plugin="${ros2_control_plugin}"
-          hw_ns="${hw_ns}" add_gripper="${add_gripper}"
+          hw_ns="${hw_ns}" add_gripper="${add_gripper}" add_bio_gripper="${add_bio_gripper}"
           robot_ip="${robot_ip}" report_type="${report_type}"
           baud_checkset="${baud_checkset}" default_gripper_baud="${default_gripper_baud}"
@@ -54,5 +55,5 @@
         <xacro:uf850_ros2_control prefix="${prefix}" velocity_control="${velocity_control}"
           ros2_control_plugin="${ros2_control_plugin}"
-          hw_ns="${hw_ns}" add_gripper="${add_gripper}"
+          hw_ns="${hw_ns}" add_gripper="${add_gripper}" add_bio_gripper="${add_bio_gripper}"
           robot_ip="${robot_ip}" report_type="${report_type}"
           baud_checkset="${baud_checkset}" default_gripper_baud="${default_gripper_baud}" />

File: src/charmie_arm_ufactory/xarm_ros2/xarm_description/urdf/xarm5/xarm5_robot_macro.xacro (robot description, xacro)
@@ -7,4 +7,5 @@
     velocity_control:=false
     add_gripper:=false
+    add_bio_gripper:=false
     ros2_control_plugin:='uf_robot_hardware/UFRobotSystemHardware'
     robot_ip:=''
@@ -29,5 +30,5 @@
           velocity_control="${velocity_control}"
           ros2_control_plugin="${ros2_control_plugin}"
-          hw_ns="${hw_ns}" add_gripper="${add_gripper}"
+          hw_ns="${hw_ns}" add_gripper="${add_gripper}" add_bio_gripper="${add_bio_gripper}"
           robot_ip="${robot_ip}" report_type="${report_type}"
           baud_checkset="${baud_checkset}" default_gripper_baud="${default_gripper_baud}"
@@ -53,5 +54,5 @@
         <xacro:xarm5_ros2_control prefix="${prefix}" velocity_control="${velocity_control}"
           ros2_control_plugin="${ros2_control_plugin}"
-          hw_ns="${hw_ns}" add_gripper="${add_gripper}"
+          hw_ns="${hw_ns}" add_gripper="${add_gripper}" add_bio_gripper="${add_bio_gripper}"
           robot_ip="${robot_ip}" report_type="${report_type}"
           baud_checkset="${baud_checkset}" default_gripper_baud="${default_gripper_baud}" />

File: src/charmie_arm_ufactory/xarm_ros2/xarm_description/urdf/xarm6/xarm6.urdf.xacro (robot description, xacro)
@@ -180,5 +180,4 @@
       <parent link="${prefix}link4"/>
       <child link="${prefix}link5"/>
-      <origin xyz="0 0 0" rpy="1.5708 0 0"/>
       <xacro:common_joint_origin joint_kinematic_params="${kinematics_params['joint5']}" />
       <axis xyz="0 0 1"/>

File: src/charmie_arm_ufactory/xarm_ros2/xarm_description/urdf/xarm6/xarm6_robot_macro.xacro (robot description, xacro)
@@ -7,4 +7,5 @@
     velocity_control:=false
     add_gripper:=false
+    add_bio_gripper:=false
     ros2_control_plugin:='uf_robot_hardware/UFRobotSystemHardware'
     robot_ip:=''
@@ -29,5 +30,5 @@
           velocity_control="${velocity_control}"
           ros2_control_plugin="${ros2_control_plugin}"
-          hw_ns="${hw_ns}" add_gripper="${add_gripper}"
+          hw_ns="${hw_ns}" add_gripper="${add_gripper}" add_bio_gripper="${add_bio_gripper}"
           robot_ip="${robot_ip}" report_type="${report_type}"
           baud_checkset="${baud_checkset}" default_gripper_baud="${default_gripper_baud}"
@@ -55,5 +56,5 @@
         <xacro:xarm6_ros2_control prefix="${prefix}" velocity_control="${velocity_control}"
           ros2_control_plugin="${ros2_control_plugin}"
-          hw_ns="${hw_ns}" add_gripper="${add_gripper}"
+          hw_ns="${hw_ns}" add_gripper="${add_gripper}" add_bio_gripper="${add_bio_gripper}"
           robot_ip="${robot_ip}" report_type="${report_type}"
           baud_checkset="${baud_checkset}" default_gripper_baud="${default_gripper_baud}" />

File: src/charmie_arm_ufactory/xarm_ros2/xarm_description/urdf/xarm7/xarm7_robot_macro.xacro (robot description, xacro)
@@ -7,4 +7,5 @@
     velocity_control:=false
     add_gripper:=false
+    add_bio_gripper:=false
     ros2_control_plugin:='uf_robot_hardware/UFRobotSystemHardware'
     robot_ip:=''
@@ -29,5 +30,5 @@
           velocity_control="${velocity_control}"
           ros2_control_plugin="${ros2_control_plugin}"
-          hw_ns="${hw_ns}" add_gripper="${add_gripper}"
+          hw_ns="${hw_ns}" add_gripper="${add_gripper}" add_bio_gripper="${add_bio_gripper}"
           robot_ip="${robot_ip}" report_type="${report_type}"
           baud_checkset="${baud_checkset}" default_gripper_baud="${default_gripper_baud}"
@@ -57,5 +58,5 @@
         <xacro:xarm7_ros2_control prefix="${prefix}" velocity_control="${velocity_control}"
           ros2_control_plugin="${ros2_control_plugin}"
-          hw_ns="${hw_ns}" add_gripper="${add_gripper}"
+          hw_ns="${hw_ns}" add_gripper="${add_gripper}" add_bio_gripper="${add_bio_gripper}"
           robot_ip="${robot_ip}" report_type="${report_type}"
           baud_checkset="${baud_checkset}" default_gripper_baud="${default_gripper_baud}" />

File: src/charmie_arm_ufactory/xarm_ros2/xarm_description/urdf/xarm_device_macro.xacro (robot description, xacro)
@@ -9,4 +9,5 @@
     add_gripper:=false
     add_vacuum_gripper:=false
+    add_bio_gripper:=false
     dof:=7
     robot_type:='xarm'
@@ -83,8 +84,8 @@
       </xacro:unless>
     </xacro:unless>
-    <xacro:if value="${robot_type == 'uf850'}">
+    <xacro:if value="${robot_type == 'uf850' or robot_type == 'xarm7_mirror'}">
       <xacro:property name="robot_name" value="${robot_type}" />
     </xacro:if>
-    <xacro:unless value="${robot_type == 'uf850'}">
+    <xacro:unless value="${robot_type == 'uf850' or robot_type == 'xarm7_mirror'}">
       <xacro:property name="robot_name" value="${robot_type}${dof}" />
     </xacro:unless>
@@ -102,4 +103,5 @@
         ros2_control_plugin="${ros2_control_plugin}"
         add_gripper="${add_gripper}"
+        add_bio_gripper="${add_bio_gripper}"
         robot_ip="${robot_ip}"
         report_type="${report_type}"
@@ -119,4 +121,5 @@
           ros2_control_plugin="${ros2_control_plugin}"
           add_gripper="${add_gripper}"
+          add_bio_gripper="${add_bio_gripper}"
           robot_ip="${robot_ip}"
           report_type="${report_type}"
@@ -150,4 +153,5 @@
           ros2_control_plugin="${ros2_control_plugin}"
           add_gripper="${add_gripper}"
+          add_bio_gripper="${add_bio_gripper}"
           robot_ip="${robot_ip}"
           report_type="${report_type}"
@@ -161,18 +165,38 @@
     </xacro:if>
     <xacro:unless value="${dof == 5 or dof == 6}">
-      <!-- Load XArm7 Robot Model URDF -->
-      <xacro:include filename="$(find xarm_description)/urdf/xarm7/xarm7_robot_macro.xacro" />
-      <xacro:xarm7_robot prefix="${prefix}" hw_ns="${hw_ns}" limited="${limited}"
-        velocity_control="${velocity_control}"
-        ros2_control_plugin="${ros2_control_plugin}"
-        add_gripper="${add_gripper}"
-        robot_ip="${robot_ip}"
-        report_type="${report_type}"
-        baud_checkset="${baud_checkset}"
-        default_gripper_baud="${default_gripper_baud}"
-        model1300="${new_model1300}"
-        inertial_params_filename="${inertial_params_filename}"
-        kinematics_params_filename="${kinematics_params_filename}"
-        hard_interface="${hard_interface}" />
+      <xacro:if value="${robot_type == 'xarm7_mirror'}">
+        <!-- Load xArm7 Mirror Robot Model URDF -->
+        <xacro:include filename="$(find xarm_description)/urdf/xarm7_mirror/xarm7_mirror_robot_macro.xacro" />
+        <xacro:xarm7_mirror_robot prefix="${prefix}" hw_ns="${hw_ns}" limited="${limited}"
+          velocity_control="${velocity_control}"
+          ros2_control_plugin="${ros2_control_plugin}"
+          add_gripper="${add_gripper}"
+          add_bio_gripper="${add_bio_gripper}"
+          robot_ip="${robot_ip}"
+          report_type="${report_type}"
+          baud_checkset="${baud_checkset}"
+          default_gripper_baud="${default_gripper_baud}"
+          model1300="${new_model1300}"
+          inertial_params_filename="${inertial_params_filename}"
+          kinematics_params_filename="${kinematics_params_filename}"
+          hard_interface="${hard_interface}" />
+      </xacro:if>
+      <xacro:unless value="${robot_type == 'xarm7_mirror'}">
+        <!-- Load XArm7 Robot Model URDF -->
+        <xacro:include filename="$(find xarm_description)/urdf/xarm7/xarm7_robot_macro.xacro" />
+        <xacro:xarm7_robot prefix="${prefix}" hw_ns="${hw_ns}" limited="${limited}"
+          velocity_control="${velocity_control}"
+          ros2_control_plugin="${ros2_control_plugin}"
+          add_gripper="${add_gripper}"
+          add_bio_gripper="${add_bio_gripper}"
+          robot_ip="${robot_ip}"
+          report_type="${report_type}"
+          baud_checkset="${baud_checkset}"
+          default_gripper_baud="${default_gripper_baud}"
+          model1300="${new_model1300}"
+          inertial_params_filename="${inertial_params_filename}"
+          kinematics_params_filename="${kinematics_params_filename}"
+          hard_interface="${hard_interface}" />
+      </xacro:unless>
     </xacro:unless>
     <xacro:if value="${add_realsense_d435i}">
@@ -206,5 +230,13 @@
       </xacro:unless>
     </xacro:if>
-    <xacro:if value="${not add_gripper and add_vacuum_gripper}">
+    <xacro:if value="${not add_gripper and add_bio_gripper}">
+      <xacro:unless value="${robot_type == 'lite'}">
+        <!-- Load BIO Gripper Model URDF -->
+        <xacro:include filename="$(find xarm_description)/urdf/gripper/bio_gripper_macro.xacro" />
+        <xacro:bio_gripper_macro prefix="${prefix}" attach_to="${prefix}link_eef"
+          ros2_control_plugin="${ros2_control_plugin}" dof="${dof}" hard_interface="${hard_interface}" />
+      </xacro:unless>
+    </xacro:if>
+    <xacro:if value="${not add_gripper and not add_bio_gripper and add_vacuum_gripper}">
       <xacro:if value="${robot_type == 'lite'}">
         <!-- Load Lite Vacuum Gripper Model URDF -->
@@ -234,8 +266,8 @@
       <xacro:include filename="$(find xarm_description)/urdf/common/common.gazebo.xacro" />
       <xacro:if value="${is_ros2}">
-        <xacro:if value="${robot_type == 'uf850'}">
+        <xacro:if value="${robot_type == 'uf850' or robot_type == 'xarm7_mirror'}">
           <xacro:property name="new_ros2_control_params" value="$(find xarm_controller)/config/${robot_type}_controllers.yaml"/>
         </xacro:if>
-        <xacro:unless value="${robot_type == 'uf850'}">
+        <xacro:unless value="${robot_type == 'uf850' or robot_type == 'xarm7_mirror'}">
           <xacro:property name="new_ros2_control_params" value="$(find xarm_controller)/config/${robot_type}${dof}_controllers.yaml"/>
         </xacro:unless>
