Commit message: Updates to simulation pre SLAM

File: src/charmie_sim/description/robot.urdf.xacro (robot description, xacro)
@@ -2,4 +2,6 @@
 <robot xmlns:xacro="http://www.ros.org/wiki/xacro"  name="robot">
     <xacro:include filename="robot_core.xacro"/>
-    <xacro:include filename="gazebo_control.xacro"/>
+    <!-- <xacro:include filename="gazebo_control.xacro"/> -->
+    <xacro:include filename="ros2_control.xacro"/>
+    <xacro:include filename="lidar.xacro"/>
 </robot>

File: src/charmie_sim/description/robot_core.xacro (robot description, xacro)
@@ -13,4 +13,7 @@
     <material name ="black">
         <color rgba="0 0 0 1" />
+    </material>
+    <material name ="red">
+        <color rgba="1 0 0 1" />
     </material>
     <!-- BASE LINK -->
@@ -60,5 +63,5 @@
         <collision>
             <geometry>
-                <cylinder radius="0.05" length="0.04"/>
+                <sphere radius="0.05"/>
             </geometry>
         </collision>
@@ -86,5 +89,5 @@
         <collision>
             <geometry>
-                <cylinder radius="0.05" length="0.04"/>
+                <sphere radius="0.05"/>
             </geometry>
         </collision>
