Commit message: Added xacro variables and functions for charmie urdf

File: src/charmie_description/urdf/charmie_.urdf.xacro (robot description, xacro)
@@ -1,4 +1,11 @@
 <?xml version="1.0"?>
 <robot name="charmie" xmlns:xacro="http://www.ros.org/wiki/xacro">
+    <xacro:property name="base_octagon_side" value="0.232" />
+    <xacro:property name="base_length" value="0.56" />
+    <xacro:property name="base_height" value="0.27" />
+    <xacro:property name="base_floor_height" value="0.05" />
+    <xacro:property name="wheel_radius" value="0.1" />
+    <xacro:property name="wheel_length" value="0.038" />
+    <xacro:property name="wheel_shift_from_base_length" value="0.025" />
     <material name ="orange">
         <color rgba="1 0.3 0.1 1" />
@@ -14,28 +21,28 @@
         <visual>
             <geometry>
-                <box size="0.56 0.235 0.27" />
+                <box size="${base_length} ${base_octagon_side} ${base_height}" />
             </geometry>
-            <origin xyz="0 0 0.135" rpy="0 0 0" />
+            <origin xyz="0 0 ${base_height/2}" rpy="0 0 0" />
             <material name="light_grey"/>
         </visual>
         <visual>
             <geometry>
-                <box size="0.56 0.235 0.27" />
+                <box size="${base_length} ${base_octagon_side} ${base_height}" />
             </geometry>
-            <origin xyz="0 0 0.135" rpy="0 0 ${pi/2}" />
+            <origin xyz="0 0 ${base_height/2}" rpy="0 0 ${pi/2}" />
             <material name="light_grey"/>
         </visual>
         <visual>
             <geometry>
-                <box size="0.56 0.235 0.27" />
+                <box size="${base_length} ${base_octagon_side} ${base_height}" />
             </geometry>
-            <origin xyz="0 0 0.135" rpy="0 0 ${pi/4}" />
+            <origin xyz="0 0 ${base_height/2}" rpy="0 0 ${pi/4}" />
             <material name="light_grey"/>
         </visual>
         <visual>
             <geometry>
-                <box size="0.56 0.235 0.27" />
+                <box size="${base_length} ${base_octagon_side} ${base_height}" />
             </geometry>
-            <origin xyz="0 0 0.135" rpy="0 0 -${pi/4}" />
+            <origin xyz="0 0 ${base_height/2}" rpy="0 0 -${pi/4}" />
             <material name="light_grey"/>
         </visual>
@@ -45,5 +52,5 @@
         <parent link="base_footprint"/>
         <child link="base_link"/>
-        <origin xyz="0 0 0.05" rpy="0 0 0"/>
+        <origin xyz="0 0 ${base_floor_height}" rpy="0 0 0"/>
     </joint>
     <link name="base_footprint">
@@ -64,46 +71,42 @@
         </visual>
     </link> -->
+    <!-- WHEEL LINK FUNCTION -->
+    <xacro:macro name="wheel_link" params="prefix">
+        <link name="${prefix}_wheel_link">
+            <visual>
+                <geometry>
+                    <cylinder radius="${wheel_radius}" length="${wheel_length}"/>
+                </geometry>
+                <origin xyz="0 0 0" rpy="${pi/2} 0 0"/>
+                <material name="black"/>
+            </visual>
+        </link>
+    </xacro:macro>
     <!-- RIGHT WHEEL -->
     <joint name="base_right_wheel_joint" type="continuous">
         <parent link="base_link"/>
         <child link="right_wheel_link"/>
-        <origin xyz="0 -0.255 0.05"/>
+        <origin xyz="0 ${-(base_length/2-wheel_shift_from_base_length)} ${wheel_radius-base_floor_height}"/>
         <axis xyz="0 1 0"/>
     </joint>
-    <link name="right_wheel_link">
-        <visual>
-            <geometry>
-                <cylinder radius="0.1" length="0.038"/>
-            </geometry>
-            <origin xyz="0 0 0" rpy="1.57 0 0"/>
-            <material name="black"/>
-        </visual>
-    </link>
+    <xacro:wheel_link prefix="right" />
     <!-- LEFT WHEEL -->
     <joint name="base_left_wheel_joint" type="continuous">
         <parent link="base_link"/>
         <child link="left_wheel_link"/>
-        <origin xyz="0 0.255 0.05"/>
+        <origin xyz="0 ${+(base_length/2-wheel_shift_from_base_length)} ${wheel_radius-base_floor_height}"/>
         <axis xyz="0 1 0"/>
     </joint>
-    <link name="left_wheel_link">
-        <visual>
-            <geometry>
-                <cylinder radius="0.1" length="0.038"/>
-            </geometry>
-            <origin xyz="0 0 0" rpy="1.57 0 0"/>
-            <material name="black"/>
-        </visual>
-    </link>
+    <xacro:wheel_link prefix="left" />
     <!-- FRONT CASTER WHEEL -->
     <joint name="base_front_caster_wheel_joint" type="fixed">
         <parent link="base_link"/>
         <child link="front_caster_wheel_link"/>
-        <origin xyz="0.255 0 -0.025"/>
+        <origin xyz="${+(base_length/2-base_floor_height/2)} 0 ${-base_floor_height/2}"/>
     </joint>
     <link name="front_caster_wheel_link">
         <visual>
             <geometry>
-                <sphere radius="0.025" />
+                <sphere radius="${base_floor_height/2}" />
             </geometry>
             <origin xyz="0 0 0" rpy="0 0 0"/>
@@ -115,10 +118,10 @@
         <parent link="base_link"/>
         <child link="back_caster_wheel_link"/>
-        <origin xyz="-0.255 0 -0.025"/>
+        <origin xyz="${-(base_length/2-base_floor_height/2)} 0 ${-base_floor_height/2}"/>
     </joint>
     <link name="back_caster_wheel_link">
         <visual>
             <geometry>
-                <sphere radius="0.025" />
+                <sphere radius="${base_floor_height/2}" />
             </geometry>
             <origin xyz="0 0 0" rpy="0 0 0"/>

Commit message: Included urdf files and added mesh files (not used for now)

File: src/charmie_description/urdf/charmie_.urdf.xacro (robot description, xacro)
@@ -1,59 +1,6 @@
 <?xml version="1.0"?>
 <robot name="charmie" xmlns:xacro="http://www.ros.org/wiki/xacro">
-    <xacro:property name="base_octagon_side" value="0.232" />
-    <xacro:property name="base_length" value="0.56" />
-    <xacro:property name="base_height" value="0.27" />
-    <xacro:property name="base_floor_height" value="0.05" />
-    <xacro:property name="wheel_radius" value="0.1" />
-    <xacro:property name="wheel_length" value="0.038" />
-    <xacro:property name="wheel_shift_from_base_length" value="0.025" />
-    <material name ="orange">
-        <color rgba="1 0.3 0.1 1" />
-    </material>
-    <material name ="black">
-        <color rgba="0 0 0 1" />
-    </material>
-    <material name ="light_grey">
-        <color rgba="0.8 0.8 0.8 1" />
-    </material>
-    <!-- BASE LINK -->
-    <link name="base_link">
-        <visual>
-            <geometry>
-                <box size="${base_length} ${base_octagon_side} ${base_height}" />
-            </geometry>
-            <origin xyz="0 0 ${base_height/2}" rpy="0 0 0" />
-            <material name="light_grey"/>
-        </visual>
-        <visual>
-            <geometry>
-                <box size="${base_length} ${base_octagon_side} ${base_height}" />
-            </geometry>
-            <origin xyz="0 0 ${base_height/2}" rpy="0 0 ${pi/2}" />
-            <material name="light_grey"/>
-        </visual>
-        <visual>
-            <geometry>
-                <box size="${base_length} ${base_octagon_side} ${base_height}" />
-            </geometry>
-            <origin xyz="0 0 ${base_height/2}" rpy="0 0 ${pi/4}" />
-            <material name="light_grey"/>
-        </visual>
-        <visual>
-            <geometry>
-                <box size="${base_length} ${base_octagon_side} ${base_height}" />
-            </geometry>
-            <origin xyz="0 0 ${base_height/2}" rpy="0 0 -${pi/4}" />
-            <material name="light_grey"/>
-        </visual>
-    </link>
-    <!-- BASE FOOTPRINT -->
-    <joint name="base_footprint_joint" type="fixed">
-        <parent link="base_footprint"/>
-        <child link="base_link"/>
-        <origin xyz="0 0 ${base_floor_height}" rpy="0 0 0"/>
-    </joint>
-    <link name="base_footprint">
-    </link>
+    <xacro:include filename="common_properties.xacro"/>
+    <xacro:include filename="mobile_base.xacro"/>
     <!-- LIDAR -->
     <!-- <joint name="lidar_joint" type="fixed">
@@ -71,61 +18,3 @@
         </visual>
     </link> -->
-    <!-- WHEEL LINK FUNCTION -->
-    <xacro:macro name="wheel_link" params="prefix">
-        <link name="${prefix}_wheel_link">
-            <visual>
-                <geometry>
-                    <cylinder radius="${wheel_radius}" length="${wheel_length}"/>
-                </geometry>
-                <origin xyz="0 0 0" rpy="${pi/2} 0 0"/>
-                <material name="black"/>
-            </visual>
-        </link>
-    </xacro:macro>
-    <!-- RIGHT WHEEL -->
-    <joint name="base_right_wheel_joint" type="continuous">
-        <parent link="base_link"/>
-        <child link="right_wheel_link"/>
-        <origin xyz="0 ${-(base_length/2-wheel_shift_from_base_length)} ${wheel_radius-base_floor_height}"/>
-        <axis xyz="0 1 0"/>
-    </joint>
-    <xacro:wheel_link prefix="right" />
-    <!-- LEFT WHEEL -->
-    <joint name="base_left_wheel_joint" type="continuous">
-        <parent link="base_link"/>
-        <child link="left_wheel_link"/>
-        <origin xyz="0 ${+(base_length/2-wheel_shift_from_base_length)} ${wheel_radius-base_floor_height}"/>
-        <axis xyz="0 1 0"/>
-    </joint>
-    <xacro:wheel_link prefix="left" />
-    <!-- FRONT CASTER WHEEL -->
-    <joint name="base_front_caster_wheel_joint" type="fixed">
-        <parent link="base_link"/>
-        <child link="front_caster_wheel_link"/>
-        <origin xyz="${+(base_length/2-base_floor_height/2)} 0 ${-base_floor_height/2}"/>
-    </joint>
-    <link name="front_caster_wheel_link">
-        <visual>
-            <geometry>
-                <sphere radius="${base_floor_height/2}" />
-            </geometry>
-            <origin xyz="0 0 0" rpy="0 0 0"/>
-            <material name="black"/>
-        </visual>
-    </link>
-    <!-- BACK CASTER WHEEL -->
-    <joint name="base_back_caster_wheel_joint" type="fixed">
-        <parent link="base_link"/>
-        <child link="back_caster_wheel_link"/>
-        <origin xyz="${-(base_length/2-base_floor_height/2)} 0 ${-base_floor_height/2}"/>
-    </joint>
-    <link name="back_caster_wheel_link">
-        <visual>
-            <geometry>
-                <sphere radius="${base_floor_height/2}" />
-            </geometry>
-            <origin xyz="0 0 0" rpy="0 0 0"/>
-            <material name="black"/>
-        </visual>
-    </link>
 </robot>

Commit message: Added inertia tags to charmie urdf

File: src/charmie_description/urdf/charmie_.urdf.xacro (robot description, xacro)
@@ -2,4 +2,5 @@
 <robot name="charmie" xmlns:xacro="http://www.ros.org/wiki/xacro">
     <xacro:include filename="common_properties.xacro"/>
+    <xacro:include filename="inertial_macros.xacro"/>
     <xacro:include filename="mobile_base.xacro"/>
     <!-- LIDAR -->

File: src/charmie_description/urdf/mobile_base.xacro (robot description, xacro)
@@ -17,4 +17,7 @@
             <material name="light_grey"/>
         </visual>
+        <xacro:inertial_box mass="5.0" x="${base_length}" y="${base_octagon_side}" z="${base_height}" >
+            <origin xyz="0 0 ${base_height/2}" rpy="0 0 0" />
+        </xacro:inertial_box>
         <visual>
             <geometry>
@@ -24,4 +27,7 @@
             <material name="light_grey"/>
         </visual>
+        <xacro:inertial_box mass="5.0" x="${base_length}" y="${base_octagon_side}" z="${base_height}" >
+            <origin xyz="0 0 ${base_height/2}" rpy="0 0 ${pi/2}" />
+        </xacro:inertial_box>
         <visual>
             <geometry>
@@ -31,4 +37,7 @@
             <material name="light_grey"/>
         </visual>
+        <xacro:inertial_box mass="5.0" x="${base_length}" y="${base_octagon_side}" z="${base_height}" >
+            <origin xyz="0 0 ${base_height/2}" rpy="0 0 ${pi/4}" />
+        </xacro:inertial_box>
         <visual>
             <geometry>
@@ -38,4 +47,7 @@
             <material name="light_grey"/>
         </visual>
+        <xacro:inertial_box mass="5.0" x="${base_length}" y="${base_octagon_side}" z="${base_height}" >
+            <origin xyz="0 0 ${base_height/2}" rpy="0 0 -${pi/4}" />
+        </xacro:inertial_box>
     </link>
     <!-- BASE FOOTPRINT -->
@@ -58,4 +70,7 @@
                 <material name="black"/>
             </visual>
+            <xacro:inertial_cylinder mass="0.5" length="${wheel_length}" radius="${wheel_radius}" >
+                <origin xyz="0 0 0" rpy="${pi/2} 0 0" />
+            </xacro:inertial_cylinder>
         </link>
     </xacro:macro>
@@ -90,4 +105,7 @@
             <material name="black"/>
         </visual>
+        <xacro:inertial_sphere mass="0.5" radius="${base_floor_height/2}" >
+            <origin xyz="0 0 0" rpy="0 0 0" />
+        </xacro:inertial_sphere>
     </link>
     <!-- BACK CASTER WHEEL -->
@@ -105,4 +123,7 @@
             <material name="black"/>
         </visual>
+        <xacro:inertial_sphere mass="0.5" radius="${base_floor_height/2}" >
+            <origin xyz="0 0 0" rpy="0 0 0" />
+        </xacro:inertial_sphere>
     </link>
 </robot>

Commit message: Added all gazebo realted charmie info (movement base), launch files and worlds

File: src/charmie_description/urdf/charmie_.urdf.xacro (robot description, xacro)
@@ -4,4 +4,5 @@
     <xacro:include filename="inertial_macros.xacro"/>
     <xacro:include filename="mobile_base.xacro"/>
+    <xacro:include filename="mobile_base_gazebo.xacro"/>
     <!-- LIDAR -->
     <!-- <joint name="lidar_joint" type="fixed">

File: src/charmie_description/urdf/mobile_base.xacro (robot description, xacro)
@@ -17,4 +17,10 @@
             <material name="light_grey"/>
         </visual>
+        <collision>
+            <geometry>
+                <box size="${base_length} ${base_octagon_side} ${base_height}" />
+            </geometry>
+            <origin xyz="0 0 ${base_height/2}" rpy="0 0 0" />
+        </collision>
         <xacro:inertial_box mass="5.0" x="${base_length}" y="${base_octagon_side}" z="${base_height}" >
             <origin xyz="0 0 ${base_height/2}" rpy="0 0 0" />
@@ -27,4 +33,10 @@
             <material name="light_grey"/>
         </visual>
+        <!-- <collision>
+            <geometry>
+                <box size="${base_length} ${base_octagon_side} ${base_height}" />
+            </geometry>
+            <origin xyz="0 0 ${base_height/2}" rpy="0 0 ${pi/2}" />
+        </collision> -->
         <xacro:inertial_box mass="5.0" x="${base_length}" y="${base_octagon_side}" z="${base_height}" >
             <origin xyz="0 0 ${base_height/2}" rpy="0 0 ${pi/2}" />
@@ -70,4 +82,10 @@
                 <material name="black"/>
             </visual>
+            <collision>
+                <geometry>
+                    <cylinder radius="${wheel_radius}" length="${wheel_length}"/>
+                </geometry>
+                <origin xyz="0 0 0" rpy="${pi/2} 0 0"/>
+            </collision>
             <xacro:inertial_cylinder mass="0.5" length="${wheel_length}" radius="${wheel_radius}" >
                 <origin xyz="0 0 0" rpy="${pi/2} 0 0" />
@@ -76,5 +94,5 @@
     </xacro:macro>
     <!-- RIGHT WHEEL -->
-    <joint name="base_right_wheel_joint" type="continuous">
+    <joint name="right_wheel_joint" type="continuous">
         <parent link="base_link"/>
         <child link="right_wheel_link"/>
@@ -84,5 +102,5 @@
     <xacro:wheel_link prefix="right" />
     <!-- LEFT WHEEL -->
-    <joint name="base_left_wheel_joint" type="continuous">
+    <joint name="left_wheel_joint" type="continuous">
         <parent link="base_link"/>
         <child link="left_wheel_link"/>
@@ -105,4 +123,10 @@
             <material name="black"/>
         </visual>
+        <collision>
+            <geometry>
+                <sphere radius="${base_floor_height/2}" />
+            </geometry>
+            <origin xyz="0 0 0" rpy="0 0 0"/>
+        </collision>
         <xacro:inertial_sphere mass="0.5" radius="${base_floor_height/2}" >
             <origin xyz="0 0 0" rpy="0 0 0" />
@@ -123,4 +147,10 @@
             <material name="black"/>
         </visual>
+        <collision>
+            <geometry>
+                <sphere radius="${base_floor_height/2}" />
+            </geometry>
+            <origin xyz="0 0 0" rpy="0 0 0"/>
+        </collision>
         <xacro:inertial_sphere mass="0.5" radius="${base_floor_height/2}" >
             <origin xyz="0 0 0" rpy="0 0 0" />

Commit message: Added hokuyo lidar to urdf

File: src/charmie_description/urdf/charmie_.urdf.xacro (robot description, xacro)
@@ -5,18 +5,4 @@
     <xacro:include filename="mobile_base.xacro"/>
     <xacro:include filename="mobile_base_gazebo.xacro"/>
-    <!-- LIDAR -->
-    <!-- <joint name="lidar_joint" type="fixed">
-        <parent link="base_link"/>
-        <child link="base_lidar"/>
-        <origin xyz="0.265 0.0 0.35"/>
-    </joint>
-    <link name="base_lidar">
-        <visual>
-            <geometry>
-                <cylinder radius="0.019" length="0.024" />
-            </geometry>
-            <origin xyz="0 0 0" rpy="0 0 0" />
-            <material name="black"/>
-        </visual>
-    </link> -->
+    <xacro:include filename="lidar.xacro"/>
 </robot>

File: src/charmie_description/urdf/mobile_base.xacro (robot description, xacro)
@@ -33,10 +33,10 @@
             <material name="light_grey"/>
         </visual>
-        <!-- <collision>
+        <collision>
             <geometry>
                 <box size="${base_length} ${base_octagon_side} ${base_height}" />
             </geometry>
             <origin xyz="0 0 ${base_height/2}" rpy="0 0 ${pi/2}" />
-        </collision> -->
+        </collision>
         <xacro:inertial_box mass="5.0" x="${base_length}" y="${base_octagon_side}" z="${base_height}" >
             <origin xyz="0 0 ${base_height/2}" rpy="0 0 ${pi/2}" />
@@ -49,4 +49,10 @@
             <material name="light_grey"/>
         </visual>
+        <collision>
+            <geometry>
+                <box size="${base_length} ${base_octagon_side} ${base_height}" />
+            </geometry>
+            <origin xyz="0 0 ${base_height/2}" rpy="0 0 ${pi/4}" />
+        </collision>
         <xacro:inertial_box mass="5.0" x="${base_length}" y="${base_octagon_side}" z="${base_height}" >
             <origin xyz="0 0 ${base_height/2}" rpy="0 0 ${pi/4}" />
@@ -59,4 +65,10 @@
             <material name="light_grey"/>
         </visual>
+        <collision>
+            <geometry>
+                <box size="${base_length} ${base_octagon_side} ${base_height}" />
+            </geometry>
+            <origin xyz="0 0 ${base_height/2}" rpy="0 0 -${pi/4}" />
+        </collision>
         <xacro:inertial_box mass="5.0" x="${base_length}" y="${base_octagon_side}" z="${base_height}" >
             <origin xyz="0 0 ${base_height/2}" rpy="0 0 -${pi/4}" />
