Commit message: Added lidar to urdf and params file for slam

File: src/charmie_description/urdf/common_properties.xacro (robot description, xacro)
@@ -10,3 +10,9 @@
         <color rgba="0.8 0.8 0.8 1" />
     </material>
+    <material name ="grey">
+        <color rgba="0.5 0.5 0.5 1" />
+    </material>
+    <material name ="dark_grey">
+        <color rgba="0.25 0.25 0.25 1" />
+    </material>
 </robot>

File: src/charmie_description/urdf/lidar.xacro (robot description, xacro)
@@ -15,5 +15,5 @@
                 <!-- <cylinder radius="0.05" length="0.04"/> -->
             </geometry>
-            <material name="black"/>
+            <material name="dark_grey"/>
         </visual>
         <collision>
