Commit message: Created 2nd node in charmie_lidar for lidar_bottom.

File: src/charmie_description/urdf/lidar_bottom.xacro (robot description, xacro)
@@ -1,10 +1,10 @@
 <?xml version="1.0"?>
 <robot xmlns:xacro="http://www.ros.org/wiki/xacro" >
-    <xacro:property name="lidar_bottom_height_from_base" value="0.1" /> <!-- 20 cm below the first lidar -->
+    <xacro:property name="lidar_bottom_height_from_base" value="0.03" /> <!-- 20 cm below the first lidar -->
     <xacro:property name="lidar_dist_from_base_limit" value="0.025" />
     <joint name="laser_bottom_joint" type="fixed">
         <parent link="base_link"/>
         <child link="lidar_bottom_frame"/>
-        <origin xyz="${(base_length/2-lidar_dist_from_base_limit)} 0 ${lidar_bottom_height_from_base}" rpy="0 0 0"/>
+        <origin xyz="${(base_length/2-lidar_dist_from_base_limit)} 0 ${lidar_bottom_height_from_base}" rpy="${pi} 0 0"/>
     </joint>
     <link name="lidar_bottom_frame">
