Commit message: Added 2nd lidar (bottom) to gazebo. Wrong coordinates.

File: src/charmie_description/urdf/charmie_gazebo.urdf.xacro (robot description, xacro)
@@ -6,4 +6,6 @@
     <xacro:include filename="mobile_base_gazebo.xacro"/>
     <xacro:include filename="lidar.xacro"/>
+    <xacro:include filename="lidar_bottom.xacro"/>
     <xacro:include filename="lidar_gazebo.xacro"/>
+    <xacro:include filename="lidar_bottom_gazebo.xacro"/>
 </robot>

File: src/charmie_description/urdf/lidar_bottom.xacro (robot description, xacro)
@@ -1,17 +1,16 @@
 <?xml version="1.0"?>
 <robot xmlns:xacro="http://www.ros.org/wiki/xacro" >
-    <xacro:property name="lidar_height_from_base" value="0.3" />
+    <xacro:property name="lidar_bottom_height_from_base" value="0.1" /> <!-- 20 cm below the first lidar -->
     <xacro:property name="lidar_dist_from_base_limit" value="0.025" />
-    <joint name="laser_joint" type="fixed">
+    <joint name="laser_bottom_joint" type="fixed">
         <parent link="base_link"/>
-        <child link="lidar_frame"/>
-        <origin xyz="${(base_length/2-lidar_dist_from_base_limit)} 0 ${lidar_height_from_base}" rpy="0 0 0"/>
+        <child link="lidar_bottom_frame"/>
+        <origin xyz="${(base_length/2-lidar_dist_from_base_limit)} 0 ${lidar_bottom_height_from_base}" rpy="0 0 0"/>
     </joint>
-    <link name="lidar_frame">
+    <link name="lidar_bottom_frame">
         <visual>
             <origin xyz="0 0 -0.062" rpy="${pi/2} 0 ${pi}"/>
             <geometry>
                 <mesh filename="file://$(find charmie_description)/meshes/lidar.stl" scale="0.001 0.001 0.001"/>
-                <!-- <cylinder radius="0.05" length="0.04"/> -->
             </geometry>
             <material name="dark_grey"/>
@@ -23,5 +22,5 @@
             </geometry>
         </collision>
-        <xacro:inertial_cylinder mass="0.1" length="0.038" radius="0.021"> <!-- ajustar -->
+        <xacro:inertial_cylinder mass="0.1" length="0.038" radius="0.021">
             <origin xyz="0 0 -0.011" rpy="0 0 0"/>
         </xacro:inertial_cylinder>

Commit message: Added first attempt oh head_camera to URDF

File: src/charmie_description/urdf/charmie_gazebo.urdf.xacro (robot description, xacro)
@@ -13,3 +13,5 @@
     <xacro:include filename="neck.xacro"/>
     <xacro:include filename="neck_gazebo.xacro"/>
+    <xacro:include filename="head_camera.xacro"/>
+    <xacro:include filename="head_camera_gazebo.xacro"/>
 </robot>

File: src/charmie_description/urdf/neck.xacro (robot description, xacro)
@@ -127,10 +127,3 @@
         </xacro:inertial_box>
     </link>
-    <joint name="head_camera_joint" type="fixed">
-        <parent link="neck_tilt_link"/>
-        <child link="head_camera_link"/>
-        <origin xyz="0.095 0.0115 0.195" rpy="0 0 0"/>
-    </joint>
-    <link name="head_camera_link">
-    </link>
 </robot>
