Commit message: Added new pkg rf2o_laser_odometry-ros2 and separated charmie_ urdf into charmie_gazebo and charmie_real

File: src/charmie_description/urdf/lidar.xacro (robot description, xacro)
@@ -27,32 +27,3 @@
         </xacro:inertial_cylinder>
     </link>
-    <!-- hokuyo -->
-    <gazebo reference="lidar_frame">
-        <material>Gazebo/Black</material>
-        <sensor type="ray" name="head_hokuyo_sensor">
-            <pose> 0 0 0 0 0 0 </pose>
-            <visualize>true</visualize>
-            <update_rate>10</update_rate>
-            <ray>
-                <scan>
-                    <horizontal>
-                        <samples>681</samples>
-                        <min_angle>-2.092387973753402</min_angle>
-                        <max_angle>2.092387973753402</max_angle>
-                    </horizontal>
-                </scan>
-                <range>
-                    <min>0.2</min>
-                    <max>5.6</max>
-                </range>
-            </ray>
-            <plugin name="laser_controller" filename="libgazebo_ros_ray_sensor.so">
-                <ros>
-                    <argument>~/out:=scan</argument>
-                </ros>
-                <output_type>sensor_msgs/LaserScan</output_type>
-                <frame_name>lidar_frame</frame_name>
-            </plugin>
-        </sensor>
-    </gazebo>
 </robot>

File: src/charmie_description/urdf/mobile_base.xacro (robot description, xacro)
@@ -77,7 +77,7 @@
     <!-- BASE FOOTPRINT -->
     <joint name="base_footprint_joint" type="fixed">
-        <parent link="base_footprint"/>
-        <child link="base_link"/>
-        <origin xyz="0 0 ${base_floor_height}" rpy="0 0 0"/>
+        <parent link="base_link"/>
+        <child link="base_footprint"/>
+        <origin xyz="0 0 ${-base_floor_height}" rpy="0 0 0"/>
     </joint>
     <link name="base_footprint">

File: src/charmie_description/urdf/mobile_base_gazebo.xacro (robot description, xacro)
@@ -20,27 +20,21 @@
         <mu2 value="0.001" />
     </gazebo>
-    <gazebo>
+    <!-- <gazebo>
         <plugin name="diff_drive" filename="libgazebo_ros_diff_drive.so">
-            <!-- Update rate in Hz -->
             <update_rate>50</update_rate>
-            <!-- Wheel Information -->
             <left_joint>left_wheel_joint</left_joint>
             <right_joint>right_wheel_joint</right_joint>
-            <!-- Kinematics -->
             <wheel_separation>0.51</wheel_separation>
             <wheel_diameter>0.2</wheel_diameter>
-            <!-- Limits -->
             <max_wheel_torque>200</max_wheel_torque>
             <max_wheel_acceleration>10.0</max_wheel_acceleration>
-            <!-- Input -->
             <command_topic>cmd_vel</command_topic>
-            <!-- Output -->
-            <odometry_topic>odom</odometry_topic>
-            <odometry_frame>odom</odometry_frame>
-            <robot_base_frame>base_footprint</robot_base_frame>
+            <odometry_topic>odom1</odometry_topic>
+            <odometry_frame>odom1</odometry_frame>
+            <robot_base_frame>base_footprint1</robot_base_frame>
             <publish_odom>true</publish_odom>
             <publish_odom_tf>true</publish_odom_tf>
             <publish_wheel_tf>true</publish_wheel_tf>
         </plugin>
-    </gazebo>
+    </gazebo> -->
 </robot>

Commit message: Fixed orientation error in lidar_top, due to parts misplacement. Now both lidars are calibrated. Also edited x position of both lidar frames.

File: src/charmie_description/urdf/lidar.xacro (robot description, xacro)
@@ -2,5 +2,5 @@
 <robot xmlns:xacro="http://www.ros.org/wiki/xacro" >
     <xacro:property name="lidar_height_from_base" value="0.3" />
-    <xacro:property name="lidar_dist_from_base_limit" value="0.025" />
+    <xacro:property name="lidar_dist_from_base_limit" value="0.015" />
     <joint name="laser_joint" type="fixed">
         <parent link="base_link"/>

File: src/charmie_description/urdf/lidar_bottom.xacro (robot description, xacro)
@@ -2,5 +2,5 @@
 <robot xmlns:xacro="http://www.ros.org/wiki/xacro" >
     <xacro:property name="lidar_bottom_height_from_base" value="0.03" /> <!-- 20 cm below the first lidar -->
-    <xacro:property name="lidar_dist_from_base_limit" value="0.025" />
+    <xacro:property name="lidar_dist_from_base_limit" value="0.035" />
     <joint name="laser_bottom_joint" type="fixed">
         <parent link="base_link"/>

Commit message: Redo to two 2D lidar architecture

File: src/charmie_description/urdf/lidar.xacro (robot description, xacro)
@@ -18,5 +18,5 @@
         </visual>
         <collision>
-            <origin xyz="0 0 -0.011" rpy="0 0 0"/>
+            <origin xyz="0 0 -0.062" rpy="0 0 0"/>
             <geometry>
                 <cylinder radius="0.021" length="0.038"/>
@@ -24,5 +24,5 @@
         </collision>
         <xacro:inertial_cylinder mass="0.1" length="0.038" radius="0.021"> <!-- ajustar -->
-            <origin xyz="0 0 -0.011" rpy="0 0 0"/>
+            <origin xyz="0 0 -0.062" rpy="0 0 0"/>
         </xacro:inertial_cylinder>
     </link>

File: src/charmie_description/urdf/lidar_bottom.xacro (robot description, xacro)
@@ -17,5 +17,5 @@
         </visual>
         <collision>
-            <origin xyz="0 0 -0.011" rpy="0 0 0"/>
+            <origin xyz="0 0 -0.062" rpy="0 0 0"/>
             <geometry>
                 <cylinder radius="0.021" length="0.038"/>
@@ -23,5 +23,5 @@
         </collision>
         <xacro:inertial_cylinder mass="0.1" length="0.038" radius="0.021">
-            <origin xyz="0 0 -0.011" rpy="0 0 0"/>
+            <origin xyz="0 0 -0.062" rpy="0 0 0"/>
         </xacro:inertial_cylinder>
     </link>
