Commit message: Added head_camera tf and plointcloud2

File: src/charmie_description/urdf/charmie_real.urdf.xacro (robot description, xacro)
@@ -8,4 +8,4 @@
     <xacro:include filename="torso.xacro"/>
     <xacro:include filename="neck.xacro"/>
-    <!-- <xacro:include filename="head_camera.xacro"/> -->
+    <xacro:include filename="head_camera.xacro"/>
 </robot>

File: src/charmie_description/urdf/common_properties.xacro (robot description, xacro)
@@ -11,5 +11,5 @@
     </material>
     <material name ="grey">
-        <color rgba="0.5 0.5 0.5 1" />
+        <color rgba="0.6 0.6 0.6 1" />
     </material>
     <material name ="dark_grey">

File: src/charmie_description/urdf/head_camera.xacro (robot description, xacro)
@@ -5,5 +5,5 @@
     <xacro:property name="neck_tilt_to_head_camera_height" value="0.195" />
     <joint name="head_camera_joint" type="fixed">
-        <parent link="legs_link"/>
+        <parent link="neck_tilt_link"/>
         <child link="head_camera_link"/>
         <origin xyz="${neck_tilt_to_head_camera_length} ${neck_tilt_to_head_camera_width} ${neck_tilt_to_head_camera_height}" rpy="0 0 0"/>

File: src/charmie_description/urdf/mobile_base.xacro (robot description, xacro)
@@ -15,5 +15,5 @@
             </geometry>
             <origin xyz="0 0 ${base_height/2}" rpy="0 0 0" />
-            <material name="light_grey"/>
+            <material name="grey"/>
         </visual>
         <collision>
@@ -31,5 +31,5 @@
             </geometry>
             <origin xyz="0 0 ${base_height/2}" rpy="0 0 ${pi/2}" />
-            <material name="light_grey"/>
+            <material name="grey"/>
         </visual>
         <collision>
@@ -47,5 +47,5 @@
             </geometry>
             <origin xyz="0 0 ${base_height/2}" rpy="0 0 ${pi/4}" />
-            <material name="light_grey"/>
+            <material name="grey"/>
         </visual>
         <collision>
@@ -63,5 +63,5 @@
             </geometry>
             <origin xyz="0 0 ${base_height/2}" rpy="0 0 -${pi/4}" />
-            <material name="light_grey"/>
+            <material name="grey"/>
         </visual>
         <collision>

Commit message: Added example for setting launch arguments for the robot URDF.

File: src/charmie_description/urdf/charmie_real.urdf.xacro (robot description, xacro)
@@ -1,4 +1,5 @@
 <?xml version="1.0"?>
 <robot name="charmie" xmlns:xacro="http://www.ros.org/wiki/xacro">
+    <xacro:arg name="wheel_radius" default="0.1"/>
     <xacro:include filename="common_properties.xacro"/>
     <xacro:include filename="inertial_macros.xacro"/>

File: src/charmie_description/urdf/mobile_base.xacro (robot description, xacro)
@@ -5,5 +5,5 @@
     <xacro:property name="base_height" value="0.27" />
     <xacro:property name="base_floor_height" value="0.05" />
-    <xacro:property name="wheel_radius" value="0.1" />
+    <xacro:property name="wheel_radius" value="$(arg wheel_radius)" />
     <xacro:property name="wheel_length" value="0.038" />
     <xacro:property name="wheel_shift_from_base_length" value="0.025" />

Commit message: Updated URDF for new temp face v2.5

File: src/charmie_description/urdf/charmie_real.urdf.xacro (robot description, xacro)
@@ -2,5 +2,5 @@
 <robot name="charmie" xmlns:xacro="http://www.ros.org/wiki/xacro">
     <xacro:arg name="wheel_radius" default="0.1"/>
-    <xacro:arg name="head_version" default="2"/>
+    <xacro:arg name="head_version" default="3"/>
     <xacro:include filename="common_properties.xacro"/>
     <xacro:include filename="inertial_macros.xacro"/>

File: src/charmie_description/urdf/face_v3.xacro (robot description, xacro)
@@ -11,19 +11,22 @@
     </joint>
     <link name="face_link">
+        <!-- Temporary adjustements (compared to older face) for updated face 2025_06 -->
+        <!-- /2 -> /2.5 -->
+        <!-- added -0.02 -->
         <visual>
-            <origin xyz="${face_length/2} 0 ${face_height_shift}" rpy="0 ${pi/2} 0"/>
+            <origin xyz="${face_length/2.5} 0 ${face_height_shift-0.02}" rpy="0 ${pi/2} 0"/>
             <geometry>
-                <cylinder radius="${face_height/2}" length="${face_length}"/>
+                <cylinder radius="${face_height/2.5}" length="${face_length}"/>
             </geometry>
             <material name="grey"/>
         </visual>
         <collision>
-            <origin xyz="${face_length/2} 0 ${face_height_shift}" rpy="0 0 0"/>
+            <origin xyz="${face_length/2.5} 0 ${face_height_shift-0.02}" rpy="0 0 0"/>
             <geometry>
-                <cylinder radius="${face_height/2}" length="${face_length}"/>
+                <cylinder radius="${face_height/2.5}" length="${face_length}"/>
             </geometry>
         </collision>
-        <xacro:inertial_cylinder mass="0.5" length="${face_length}" radius="${face_height/2}" >
-            <origin xyz="${face_length/2} 0 ${face_height_shift}" rpy="0 0 0"/>
+        <xacro:inertial_cylinder mass="0.5" length="${face_length}" radius="${face_height/2.5}" >
+            <origin xyz="${face_length/2.5} 0 ${face_height_shift-0.02}" rpy="0 0 0"/>
         </xacro:inertial_cylinder>
     </link>

File: src/charmie_description/urdf/head_camera.xacro (robot description, xacro)
@@ -6,8 +6,12 @@
     <xacro:property name="head_camera_width" value="0.145" />
     <xacro:property name="head_camera_height" value="0.052" />
+    <!-- Temporary adjustements (compared to older face) for updated face 2025_06 -->
+    <xacro:property name="adjust_for_temp_face_x" value="0.0045" />
+    <xacro:property name="adjust_for_temp_face_y" value="0.0" />
+    <xacro:property name="adjust_for_temp_face_z" value="-0.075" />
     <joint name="head_camera_joint" type="fixed">
         <parent link="face_link"/>
         <child link="head_camera_link"/>
-        <origin xyz="${camera_dist_from_face_link} 0 ${camera_height_from_face_link}" rpy="0 0 0"/>
+        <origin xyz="${camera_dist_from_face_link+adjust_for_temp_face_x} 0 ${camera_height_from_face_link+adjust_for_temp_face_z}" rpy="0 0 0"/>
     </joint>
     <link name="head_camera_link">

Commit message: Added livoxmid360 3D lidar to URDF and created TF

File: src/charmie_description/urdf/charmie_real.urdf.xacro (robot description, xacro)
@@ -8,4 +8,5 @@
     <xacro:include filename="lidar.xacro"/>
     <xacro:include filename="lidar_bottom.xacro"/>
+    <xacro:include filename="lidar3d_livox_mid360.xacro"/>
     <xacro:include filename="torso.xacro"/>
     <xacro:include filename="neck.xacro"/>

File: src/charmie_description/urdf/lidar.xacro (robot description, xacro)
@@ -13,5 +13,4 @@
             <geometry>
                 <mesh filename="file://$(find charmie_description)/meshes/lidar.stl" scale="0.001 0.001 0.001"/>
-                <!-- <cylinder radius="0.05" length="0.04"/> -->
             </geometry>
             <material name="dark_grey"/>
@@ -23,5 +22,5 @@
             </geometry>
         </collision>
-        <xacro:inertial_cylinder mass="0.1" length="0.038" radius="0.021"> <!-- ajustar -->
+        <xacro:inertial_cylinder mass="0.1" length="0.038" radius="0.021">
             <origin xyz="0 0 -0.062" rpy="0 0 0"/>
         </xacro:inertial_cylinder>

File: src/charmie_description/urdf/lidar3d_livox_mid360.xacro (robot description, xacro)
@@ -1,12 +1,12 @@
 <?xml version="1.0"?>
 <robot xmlns:xacro="http://www.ros.org/wiki/xacro" >
-    <xacro:property name="lidar_bottom_height_from_base" value="0.03" />
-    <xacro:property name="lidar_bottom_dist_from_base_limit" value="0.035" />
-    <joint name="laser_bottom_joint" type="fixed">
+    <xacro:property name="lidar_livox_height_from_base" value="0.375" />
+    <xacro:property name="lidar_livox_dist_from_base_limit" value="0.065" />
+    <joint name="laser_livox_joint" type="fixed">
         <parent link="base_link"/>
-        <child link="lidar_bottom_frame"/>
-        <origin xyz="${(base_length/2-lidar_bottom_dist_from_base_limit)} 0 ${lidar_bottom_height_from_base}" rpy="${pi} 0 0"/>
+        <child link="lidar_livox_frame"/>
+        <origin xyz="${(base_length/2-lidar_livox_dist_from_base_limit)} 0 ${lidar_livox_height_from_base}" rpy="0 0 ${-pi/2}"/>
     </joint>
-    <link name="lidar_bottom_frame">
+    <link name="lidar_livox_frame">
         <visual>
             <origin xyz="0 0 -0.062" rpy="${pi/2} 0 ${pi}"/>
