Commit message: Added livox mid360 .stl mesh to livox xacro

File: src/charmie_description/urdf/lidar3d_livox_mid360.xacro (robot description, xacro)
@@ -10,12 +10,12 @@
     <link name="lidar_livox_frame">
         <visual>
-            <origin xyz="0 0 -0.062" rpy="${pi/2} 0 ${pi}"/>
+            <origin xyz="0 0 -0.02" rpy="${pi/2} 0 ${pi}"/>
             <geometry>
-                <mesh filename="file://$(find charmie_description)/meshes/lidar.stl" scale="0.001 0.001 0.001"/>
+                <mesh filename="file://$(find charmie_description)/meshes/livox_mid_360.stl" scale="0.001 0.001 0.001"/>
             </geometry>
             <material name="dark_grey"/>
         </visual>
         <collision>
-            <origin xyz="0 0 -0.062" rpy="0 0 0"/>
+            <origin xyz="0 0 -0.02" rpy="0 0 0"/>
             <geometry>
                 <cylinder radius="0.021" length="0.038"/>
@@ -23,5 +23,5 @@
         </collision>
         <xacro:inertial_cylinder mass="0.1" length="0.038" radius="0.021">
-            <origin xyz="0 0 -0.062" rpy="0 0 0"/>
+            <origin xyz="0 0 -0.02" rpy="0 0 0"/>
         </xacro:inertial_cylinder>
     </link>

Commit message: Calibrated lixox_frame TF

File: src/charmie_description/urdf/lidar3d_livox_mid360.xacro (robot description, xacro)
@@ -1,14 +1,14 @@
 <?xml version="1.0"?>
 <robot xmlns:xacro="http://www.ros.org/wiki/xacro" >
-    <xacro:property name="lidar_livox_height_from_base" value="0.375" />
+    <xacro:property name="lidar_livox_height_from_base" value="0.335" />
     <xacro:property name="lidar_livox_dist_from_base_limit" value="0.065" />
     <joint name="laser_livox_joint" type="fixed">
         <parent link="base_link"/>
-        <child link="lidar_livox_frame"/>
+        <child link="livox_frame"/>
         <origin xyz="${(base_length/2-lidar_livox_dist_from_base_limit)} 0 ${lidar_livox_height_from_base}" rpy="0 0 ${-pi/2}"/>
     </joint>
-    <link name="lidar_livox_frame">
+    <link name="livox_frame">
         <visual>
-            <origin xyz="0 0 -0.02" rpy="${pi/2} 0 ${pi}"/>
+            <origin xyz="0 0 0.025" rpy="${pi/2} 0 ${pi}"/>
             <geometry>
                 <mesh filename="file://$(find charmie_description)/meshes/livox_mid_360.stl" scale="0.001 0.001 0.001"/>
@@ -17,5 +17,5 @@
         </visual>
         <collision>
-            <origin xyz="0 0 -0.02" rpy="0 0 0"/>
+            <origin xyz="0 0 0.025" rpy="0 0 0"/>
             <geometry>
                 <cylinder radius="0.021" length="0.038"/>
@@ -23,5 +23,5 @@
         </collision>
         <xacro:inertial_cylinder mass="0.1" length="0.038" radius="0.021">
-            <origin xyz="0 0 -0.02" rpy="0 0 0"/>
+            <origin xyz="0 0 0.025" rpy="0 0 0"/>
         </xacro:inertial_cylinder>
     </link>
