Commit message: Updated lidars and base_camera position in urdf so that all obstacles detection are matching in 3D space

File: src/charmie_description/urdf/base_camera.xacro (robot description, xacro)
@@ -1,6 +1,6 @@
 <?xml version="1.0"?>
 <robot xmlns:xacro="http://www.ros.org/wiki/xacro" >
-    <xacro:property name="camera_height_from_base" value="0.4" />
-    <xacro:property name="camera_dist_from_base_limit" value="0.0" />
+    <xacro:property name="camera_height_from_base" value="0.25" />
+    <xacro:property name="camera_dist_from_base_limit" value="0.01" />
     <xacro:property name="base_camera_length" value="0.04" />
     <xacro:property name="base_camera_width" value="0.165" />
@@ -9,5 +9,5 @@
         <parent link="base_link"/>
         <child link="base_camera_link"/>
-        <origin xyz="${(base_length/2-camera_dist_from_base_limit)} 0 ${camera_height_from_base}" rpy="0 0 0"/>
+        <origin xyz="${(base_length/2-camera_dist_from_base_limit)} -0.05 ${camera_height_from_base}" rpy="0 0 0.1"/>
     </joint>
     <link name="base_camera_link">

File: src/charmie_description/urdf/lidar.xacro (robot description, xacro)
@@ -1,5 +1,5 @@
 <?xml version="1.0"?>
 <robot xmlns:xacro="http://www.ros.org/wiki/xacro" >
-    <xacro:property name="lidar_height_from_base" value="0.3" />
+    <xacro:property name="lidar_height_from_base" value="0.34" />
     <xacro:property name="lidar_dist_from_base_limit" value="0.015" />
     <joint name="laser_joint" type="fixed">

Commit message: Calibrated head camera point cloud to match the two lidars and base_camera

File: src/charmie_description/urdf/base_camera.xacro (robot description, xacro)
@@ -9,5 +9,5 @@
         <parent link="base_link"/>
         <child link="base_camera_link"/>
-        <origin xyz="${(base_length/2-camera_dist_from_base_limit)} -0.05 ${camera_height_from_base}" rpy="0 0 0.1"/>
+        <origin xyz="${(base_length/2-camera_dist_from_base_limit)} -0.05 ${camera_height_from_base}" rpy="0 0 0.05"/>
     </joint>
     <link name="base_camera_link">

File: src/charmie_description/urdf/neck.xacro (robot description, xacro)
@@ -41,5 +41,5 @@
             </geometry>
         </collision>
-        <xacro:inertial_box mass="2.0" x="${neck_pan_length}" y="${neck_pan_width}" z="${legs_height}" >
+        <xacro:inertial_box mass="2.0" x="${neck_pan_length}" y="${neck_pan_width}" z="${-neck_pan_height/2}" >
             <origin xyz="${-servo_center_to_rotation_axis} 0 ${-neck_pan_height/2}" rpy="0 0 0" />
         </xacro:inertial_box>

Commit message: Fixed visual frame for base_camera

File: src/charmie_description/urdf/base_camera.xacro (robot description, xacro)
@@ -6,12 +6,14 @@
     <xacro:property name="base_camera_width" value="0.165" />
     <xacro:property name="base_camera_height" value="0.03" />
+    <xacro:property name="yy_shift_for_optical_frame" value="-0.05" />
+    <xacro:property name="yaw_shift_for_optical_frame" value="-0.05" />
     <joint name="base_camera_joint" type="fixed">
         <parent link="base_link"/>
         <child link="base_camera_link"/>
-        <origin xyz="${(base_length/2-camera_dist_from_base_limit)} -0.05 ${camera_height_from_base}" rpy="0 0 0.05"/>
+        <origin xyz="${(base_length/2-camera_dist_from_base_limit)} ${yy_shift_for_optical_frame} ${camera_height_from_base}" rpy="0 0 ${yaw_shift_for_optical_frame}"/>
     </joint>
     <link name="base_camera_link">
         <visual>
-            <origin xyz="${-head_camera_length/2} 0 0" rpy="0 0 0"/>
+            <origin xyz="${-head_camera_length/2} ${-yy_shift_for_optical_frame} 0" rpy="0 0 ${-yaw_shift_for_optical_frame}"/>
             <geometry>
                 <box size="${head_camera_length} ${head_camera_width} ${head_camera_height}" />
@@ -20,5 +22,5 @@
         </visual>
         <collision>
-            <origin xyz="${-head_camera_length/2} 0 0" rpy="0 0 0"/>
+            <origin xyz="${-head_camera_length/2} ${-yy_shift_for_optical_frame} 0" rpy="0 0 ${-yaw_shift_for_optical_frame}"/>
             <geometry>
                 <box size="${head_camera_length} ${head_camera_width} ${head_camera_height}" />
@@ -26,5 +28,5 @@
         </collision>
         <xacro:inertial_box mass="0.5" x="${head_camera_length}" y="${head_camera_width}" z="${head_camera_height}" >
-            <origin xyz="${-head_camera_length/2} 0 0" rpy="0 0 0"/>
+            <origin xyz="${-head_camera_length/2} ${-yy_shift_for_optical_frame} 0" rpy="0 0 ${-yaw_shift_for_optical_frame}"/>
         </xacro:inertial_box>
     </link>

Commit message: Fixed hand camera transforms. Fixed object_detrections camera frames. Fixed base_camera wrong direction for yaw adjustement.

File: src/charmie_description/urdf/base_camera.xacro (robot description, xacro)
@@ -7,5 +7,5 @@
     <xacro:property name="base_camera_height" value="0.03" />
     <xacro:property name="yy_shift_for_optical_frame" value="-0.05" />
-    <xacro:property name="yaw_shift_for_optical_frame" value="-0.05" />
+    <xacro:property name="yaw_shift_for_optical_frame" value="0.05" />
     <joint name="base_camera_joint" type="fixed">
         <parent link="base_link"/>

Commit message: Updated robot URDF separating neck, face and head_camera, into individual xacros.

File: src/charmie_description/urdf/base_camera.xacro (robot description, xacro)
@@ -15,18 +15,18 @@
     <link name="base_camera_link">
         <visual>
-            <origin xyz="${-head_camera_length/2} ${-yy_shift_for_optical_frame} 0" rpy="0 0 ${-yaw_shift_for_optical_frame}"/>
+            <origin xyz="${-base_camera_length/2} ${-yy_shift_for_optical_frame} 0" rpy="0 0 ${-yaw_shift_for_optical_frame}"/>
             <geometry>
-                <box size="${head_camera_length} ${head_camera_width} ${head_camera_height}" />
+                <box size="${base_camera_length} ${base_camera_width} ${base_camera_height}" />
             </geometry>
             <material name="grey"/>
         </visual>
         <collision>
-            <origin xyz="${-head_camera_length/2} ${-yy_shift_for_optical_frame} 0" rpy="0 0 ${-yaw_shift_for_optical_frame}"/>
+            <origin xyz="${-base_camera_length/2} ${-yy_shift_for_optical_frame} 0" rpy="0 0 ${-yaw_shift_for_optical_frame}"/>
             <geometry>
-                <box size="${head_camera_length} ${head_camera_width} ${head_camera_height}" />
+                <box size="${base_camera_length} ${base_camera_width} ${base_camera_height}" />
             </geometry>
         </collision>
-        <xacro:inertial_box mass="0.5" x="${head_camera_length}" y="${head_camera_width}" z="${head_camera_height}" >
-            <origin xyz="${-head_camera_length/2} ${-yy_shift_for_optical_frame} 0" rpy="0 0 ${-yaw_shift_for_optical_frame}"/>
+        <xacro:inertial_box mass="0.5" x="${base_camera_length}" y="${base_camera_width}" z="${base_camera_height}" >
+            <origin xyz="${-base_camera_length/2} ${-yy_shift_for_optical_frame} 0" rpy="0 0 ${-yaw_shift_for_optical_frame}"/>
         </xacro:inertial_box>
     </link>

File: src/charmie_description/urdf/charmie_gazebo.urdf.xacro (robot description, xacro)
@@ -13,4 +13,5 @@
     <xacro:include filename="neck.xacro"/>
     <xacro:include filename="neck_gazebo.xacro"/>
+    <xacro:include filename="face_v2.xacro"/>
     <xacro:include filename="head_camera.xacro"/>
     <xacro:include filename="head_camera_gazebo.xacro"/>

File: src/charmie_description/urdf/charmie_real.urdf.xacro (robot description, xacro)
@@ -9,4 +9,5 @@
     <xacro:include filename="torso.xacro"/>
     <xacro:include filename="neck.xacro"/>
+    <xacro:include filename="face_v3.xacro"/>
     <xacro:include filename="head_camera.xacro"/>
     <xacro:include filename="base_camera.xacro"/>

File: src/charmie_description/urdf/hand_camera.xacro (robot description, xacro)
@@ -1,6 +1,6 @@
 <?xml version="1.0"?>
 <robot xmlns:xacro="http://www.ros.org/wiki/xacro" >
-    <xacro:property name="camera_height_from_base" value="0.25" />
-    <xacro:property name="camera_dist_from_base_limit" value="0.01" />
+    <xacro:property name="camera_dist_from_top_torso" value="0.01" />
+    <xacro:property name="camera_height_from_top_torso" value="0.25" />
     <xacro:property name="hand_camera_length" value="0.023" />
     <xacro:property name="hand_camera_width" value="0.042" />
@@ -9,5 +9,5 @@
         <parent link="top_torso_link"/>
         <child link="hand_camera_link"/>
-        <origin xyz="${(base_length/2-camera_dist_from_base_limit)} 0 ${camera_height_from_base}" rpy="0 0 0"/>
+        <origin xyz="${(base_length/2-camera_dist_from_top_torso)} 0 ${camera_height_from_top_torso}" rpy="0 0 0"/>
     </joint>
     <link name="hand_camera_link">

File: src/charmie_description/urdf/head_camera.xacro (robot description, xacro)
@@ -1,27 +1,31 @@
 <?xml version="1.0"?>
 <robot xmlns:xacro="http://www.ros.org/wiki/xacro" >
-    <xacro:property name="neck_tilt_to_head_camera_length" value="0.095" />
-    <xacro:property name="neck_tilt_to_head_camera_width" value="0.0115" />
-    <xacro:property name="neck_tilt_to_head_camera_height" value="0.195" />
+    <xacro:property name="camera_dist_from_face_link" value="${face_length + head_camera_length}" />
+    <xacro:property name="camera_height_from_face_link" value="${face_height_shift+face_height/2-head_camera_height/2-0.008}" />
+    <xacro:property name="head_camera_length" value="0.034" />
+    <xacro:property name="head_camera_width" value="0.145" />
+    <xacro:property name="head_camera_height" value="0.052" />
     <joint name="head_camera_joint" type="fixed">
-        <parent link="neck_tilt_link"/>
+        <parent link="face_link"/>
         <child link="head_camera_link"/>
-        <origin xyz="${neck_tilt_to_head_camera_length} ${neck_tilt_to_head_camera_width} ${neck_tilt_to_head_camera_height}" rpy="0 0 0"/>
+        <origin xyz="${camera_dist_from_face_link} 0 ${camera_height_from_face_link}" rpy="0 0 0"/>
     </joint>
     <link name="head_camera_link">
-        <!-- <visual>
-            <origin xyz="0 0 0" rpy="0 0 0"/>
+        <visual>
+            <origin xyz="${-head_camera_length/2} 0 0" rpy="0 0 0"/>
             <geometry>
-                <box size="0.1 0.1 0.1" />
+                <box size="${head_camera_length} ${head_camera_width} ${head_camera_height}" />
             </geometry>
             <material name="grey"/>
-        </visual> -->
-    </link>
-    <joint name="head_camera_optical_joint" type="fixed">
-        <parent link="head_camera_link"/>
-        <child link="head_camera_optical_link"/>
-        <origin xyz="0 0 0" rpy="${-pi/2} 0 ${-pi/2}"/>
-    </joint>
-    <link name="head_camera_optical_link">
+        </visual>
+        <collision>
+            <origin xyz="${-head_camera_length/2} 0 0" rpy="0 0 0"/>
+            <geometry>
+                <box size="${head_camera_length} ${head_camera_width} ${head_camera_height}" />
+            </geometry>
+        </collision>
+        <xacro:inertial_box mass="0.5" x="${head_camera_length}" y="${head_camera_width}" z="${head_camera_height}" >
+            <origin xyz="${-head_camera_length/2} 0 0" rpy="0 0 0"/>
+        </xacro:inertial_box>
     </link>
 </robot>

File: src/charmie_description/urdf/neck.xacro (robot description, xacro)
@@ -14,12 +14,4 @@
     <xacro:property name="neck_tilt_shaft_width" value="0.051" />
     <xacro:property name="neck_tilt_shaft_height" value="0.028" />
-    <xacro:property name="face_length" value="0.013" />
-    <xacro:property name="face_width" value="0.16" />
-    <xacro:property name="face_height" value="0.26" />
-    <xacro:property name="face_height_shift" value="0.0975" />
-    <xacro:property name="head_camera_length" value="0.034" />
-    <xacro:property name="head_camera_width" value="0.145" />
-    <xacro:property name="head_camera_height" value="0.052" />
-    <xacro:property name="head_camera_height_shift" value="0.0975" />
     <joint name="neck_base" type="fixed">
         <parent link="top_torso_link"/>
@@ -94,36 +86,4 @@
             <origin xyz="${neck_tilt_shaft_length/2} 0 0" rpy="0 0 0"/>
         </xacro:inertial_box>
-        <visual>
-            <origin xyz="${neck_tilt_shaft_length + face_length/2} 0 ${face_height_shift}" rpy="0 0 0"/>
-            <geometry>
-                <box size="${face_length} ${face_width} ${face_height}" />
-            </geometry>
-            <material name="grey"/>
-        </visual>
-        <collision>
-            <origin xyz="${neck_tilt_shaft_length + face_length/2} 0 ${face_height_shift}" rpy="0 0 0"/>
-            <geometry>
-                <box size="${face_length} ${face_width} ${face_height}" />
-            </geometry>
-        </collision>
-        <xacro:inertial_box mass="0.5" x="${face_length}" y="${face_width}" z="${face_height}" >
-            <origin xyz="${neck_tilt_shaft_length + face_length/2} 0 ${face_height_shift}" rpy="0 0 0"/>
-        </xacro:inertial_box>
-        <visual>
-            <origin xyz="${neck_tilt_shaft_length + face_length + head_camera_length/2} 0 ${face_height_shift+face_height/2-head_camera_height/2-0.008}" rpy="0 0 0"/>
-            <geometry>
-                <box size="${head_camera_length} ${head_camera_width} ${head_camera_height}" />
-            </geometry>
-            <material name="grey"/>
-        </visual>
-        <collision>
-            <origin xyz="${neck_tilt_shaft_length + face_length/2} 0 ${face_height_shift}" rpy="0 0 0"/>
-            <geometry>
-                <box size="${head_camera_length} ${head_camera_width} ${head_camera_height}" />
-            </geometry>
-        </collision>
-        <xacro:inertial_box mass="0.5" x="${head_camera_length}" y="${head_camera_width}" z="${head_camera_height}" >
-            <origin xyz="${neck_tilt_shaft_length + face_length/2} 0 ${face_height_shift}" rpy="0 0 0"/>
-        </xacro:inertial_box>
     </link>
 </robot>

Commit message: Updated base_camera URDF for 20 degrees down rotation

File: src/charmie_description/urdf/base_camera.xacro (robot description, xacro)
@@ -8,8 +8,9 @@
     <xacro:property name="yy_shift_for_optical_frame" value="-0.05" />
     <xacro:property name="yaw_shift_for_optical_frame" value="0.05" />
+    <xacro:property name="twenty_degrees_down_rotation" value="0.34906585" />
     <joint name="base_camera_joint" type="fixed">
         <parent link="base_link"/>
         <child link="base_camera_link"/>
-        <origin xyz="${(base_length/2-camera_dist_from_base_limit)} ${yy_shift_for_optical_frame} ${camera_height_from_base}" rpy="0 0 ${yaw_shift_for_optical_frame}"/>
+        <origin xyz="${(base_length/2-camera_dist_from_base_limit)} ${yy_shift_for_optical_frame} ${camera_height_from_base}" rpy="0 ${twenty_degrees_down_rotation} ${yaw_shift_for_optical_frame}"/>
     </joint>
     <link name="base_camera_link">

Commit message: Recalibrated yaw and yy shift for base_camera TF

File: src/charmie_description/urdf/base_camera.xacro (robot description, xacro)
@@ -6,6 +6,6 @@
     <xacro:property name="base_camera_width" value="0.165" />
     <xacro:property name="base_camera_height" value="0.03" />
-    <xacro:property name="yy_shift_for_optical_frame" value="-0.05" />
-    <xacro:property name="yaw_shift_for_optical_frame" value="0.05" />
+    <xacro:property name="yy_shift_for_optical_frame" value="0.00" />
+    <xacro:property name="yaw_shift_for_optical_frame" value="0.00" />
     <xacro:property name="twenty_degrees_down_rotation" value="0.34906585" />
     <joint name="base_camera_joint" type="fixed">

Commit message: Recalibrated base_camera and lidar_top TFs (height)

File: src/charmie_description/urdf/base_camera.xacro (robot description, xacro)
@@ -1,5 +1,5 @@
 <?xml version="1.0"?>
 <robot xmlns:xacro="http://www.ros.org/wiki/xacro" >
-    <xacro:property name="camera_height_from_base" value="0.25" />
+    <xacro:property name="camera_height_from_base" value="0.215" />
     <xacro:property name="camera_dist_from_base_limit" value="0.01" />
     <xacro:property name="base_camera_length" value="0.04" />

File: src/charmie_description/urdf/lidar.xacro (robot description, xacro)
@@ -1,5 +1,5 @@
 <?xml version="1.0"?>
 <robot xmlns:xacro="http://www.ros.org/wiki/xacro" >
-    <xacro:property name="lidar_height_from_base" value="0.34" />
+    <xacro:property name="lidar_height_from_base" value="0.31" />
     <xacro:property name="lidar_dist_from_base_limit" value="0.015" />
     <joint name="laser_joint" type="fixed">

Commit message: Merge "main" into "ObjectGrabTest" branch

File: src/charmie_description/urdf/base_camera.xacro (robot description, xacro)
@@ -1,15 +1,16 @@
 <?xml version="1.0"?>
 <robot xmlns:xacro="http://www.ros.org/wiki/xacro" >
-    <xacro:property name="camera_height_from_base" value="0.25" />
+    <xacro:property name="camera_height_from_base" value="0.215" />
     <xacro:property name="camera_dist_from_base_limit" value="0.01" />
     <xacro:property name="base_camera_length" value="0.04" />
     <xacro:property name="base_camera_width" value="0.165" />
     <xacro:property name="base_camera_height" value="0.03" />
-    <xacro:property name="yy_shift_for_optical_frame" value="-0.05" />
-    <xacro:property name="yaw_shift_for_optical_frame" value="0.05" />
+    <xacro:property name="yy_shift_for_optical_frame" value="0.00" />
+    <xacro:property name="yaw_shift_for_optical_frame" value="0.00" />
+    <xacro:property name="twenty_degrees_down_rotation" value="0.34906585" />
     <joint name="base_camera_joint" type="fixed">
         <parent link="base_link"/>
         <child link="base_camera_link"/>
-        <origin xyz="${(base_length/2-camera_dist_from_base_limit)} ${yy_shift_for_optical_frame} ${camera_height_from_base}" rpy="0 0 ${yaw_shift_for_optical_frame}"/>
+        <origin xyz="${(base_length/2-camera_dist_from_base_limit)} ${yy_shift_for_optical_frame} ${camera_height_from_base}" rpy="0 ${twenty_degrees_down_rotation} ${yaw_shift_for_optical_frame}"/>
     </joint>
     <link name="base_camera_link">

File: src/charmie_description/urdf/lidar.xacro (robot description, xacro)
@@ -1,5 +1,5 @@
 <?xml version="1.0"?>
 <robot xmlns:xacro="http://www.ros.org/wiki/xacro" >
-    <xacro:property name="lidar_height_from_base" value="0.34" />
+    <xacro:property name="lidar_height_from_base" value="0.31" />
     <xacro:property name="lidar_dist_from_base_limit" value="0.015" />
     <joint name="laser_joint" type="fixed">
@@ -13,16 +13,15 @@
             <geometry>
                 <mesh filename="file://$(find charmie_description)/meshes/lidar.stl" scale="0.001 0.001 0.001"/>
-                <!-- <cylinder radius="0.05" length="0.04"/> -->
             </geometry>
             <material name="dark_grey"/>
         </visual>
         <collision>
-            <origin xyz="0 0 -0.011" rpy="0 0 0"/>
+            <origin xyz="0 0 -0.062" rpy="0 0 0"/>
             <geometry>
                 <cylinder radius="0.021" length="0.038"/>
             </geometry>
         </collision>
-        <xacro:inertial_cylinder mass="0.1" length="0.038" radius="0.021"> <!-- ajustar -->
-            <origin xyz="0 0 -0.011" rpy="0 0 0"/>
+        <xacro:inertial_cylinder mass="0.1" length="0.038" radius="0.021">
+            <origin xyz="0 0 -0.062" rpy="0 0 0"/>
         </xacro:inertial_cylinder>
     </link>

File: src/charmie_description/urdf/lidar_bottom.xacro (robot description, xacro)
@@ -1,10 +1,10 @@
 <?xml version="1.0"?>
 <robot xmlns:xacro="http://www.ros.org/wiki/xacro" >
-    <xacro:property name="lidar_bottom_height_from_base" value="0.03" /> <!-- 20 cm below the first lidar -->
-    <xacro:property name="lidar_dist_from_base_limit" value="0.035" />
+    <xacro:property name="lidar_bottom_height_from_base" value="0.03" />
+    <xacro:property name="lidar_bottom_dist_from_base_limit" value="0.035" />
     <joint name="laser_bottom_joint" type="fixed">
         <parent link="base_link"/>
         <child link="lidar_bottom_frame"/>
-        <origin xyz="${(base_length/2-lidar_dist_from_base_limit)} 0 ${lidar_bottom_height_from_base}" rpy="${pi} 0 0"/>
+        <origin xyz="${(base_length/2-lidar_bottom_dist_from_base_limit)} 0 ${lidar_bottom_height_from_base}" rpy="${pi} 0 0"/>
     </joint>
     <link name="lidar_bottom_frame">
@@ -17,5 +17,5 @@
         </visual>
         <collision>
-            <origin xyz="0 0 -0.011" rpy="0 0 0"/>
+            <origin xyz="0 0 -0.062" rpy="0 0 0"/>
             <geometry>
                 <cylinder radius="0.021" length="0.038"/>
@@ -23,5 +23,5 @@
         </collision>
         <xacro:inertial_cylinder mass="0.1" length="0.038" radius="0.021">
-            <origin xyz="0 0 -0.011" rpy="0 0 0"/>
+            <origin xyz="0 0 -0.062" rpy="0 0 0"/>
         </xacro:inertial_cylinder>
     </link>
