Commit message: Fixed Arm Links Meshes Errors

File: src/charmie_description/urdf/arm.xacro (robot description, xacro)
@@ -4,10 +4,11 @@
   <xacro:property name="is_ros2" value="true"/>
   <xacro:property name="use_xacro_load_yaml" value="true"/>
-  <xacro:property name="mesh_path" value="xarm_description/meshes"/>
-  <xacro:property name="mesh_suffix" value=".STL"/>
+  <xacro:property name="mesh_path" value="package://xarm_description/meshes"/>
+  <xacro:property name="mesh_suffix" value="stl"/>
   <xacro:property name="kinematics_params_file" value="$(find xarm_description)/config/kinematics/default/xarm6_default_kinematics.yaml"/>
   <!-- Include xArm6 macro definition -->
   <xacro:include filename="$(find xarm_description)/urdf/xarm6/xarm6_robot_macro.xacro" />
   <xacro:include filename="$(find xarm_description)/urdf/common/common.link.xacro" />
+  <xacro:include filename="$(find xarm_description)/urdf/common/common.material.xacro" />
   <!-- Instantiate the xArm6 robot with a safe prefix -->
   <xacro:xarm6_robot
@@ -32,5 +33,5 @@
     <child link="xarm_link_base"/>
     <!-- Adjust this origin if needed for proper placement -->
-    <origin xyz="0.0 0.0 0.0" rpy="-${pi/2} 0 0"/>
+    <origin xyz="-0.12 0.06 -0.09" rpy="${pi/2} 0 0"/>
   </joint>
 </robot>

Commit message: Arm orientation and position adjustment w/o hand camera

File: src/charmie_description/urdf/arm.xacro (robot description, xacro)
@@ -6,4 +6,6 @@
   <xacro:property name="mesh_path" value="package://xarm_description/meshes"/>
   <xacro:property name="mesh_suffix" value="stl"/>
+  <!--<xacro:property name="torso_initial_angle_rads" value="0.15708" />-->
+  <xacro:property name="torso_initial_angle_rads" value="0"/>
   <xacro:property name="kinematics_params_file" value="$(find xarm_description)/config/kinematics/default/xarm6_default_kinematics.yaml"/>
   <!-- Include xArm6 macro definition -->
@@ -38,5 +40,5 @@
     <child link="xarm_link_base"/>
     <!-- Adjust this origin if needed for proper placement -->
-    <origin xyz="-0.12 0.06 -0.09" rpy="${pi/2} ${pi} 0"/>
+    <origin xyz="-0.11 0.0585 -0.0623" rpy="${pi/2} ${pi+torso_initial_angle_rads} 0"/>
   </joint>
 </robot>

Commit message: Made some necessary changes to arm.xacro and to some moveit config files

File: src/charmie_description/urdf/arm.xacro (robot description, xacro)
@@ -1,4 +1,6 @@
 <?xml version="1.0"?>
 <robot xmlns:xacro="http://www.ros.org/wiki/xacro">
+  <!-- Add argument for hardware selection -->
+  <xacro:arg name="use_real_hardware" default="false"/>
   <!-- Set required flags used by xarm_description flags -->
   <xacro:property name="is_ros2" value="true"/>
@@ -23,4 +25,14 @@
   <xacro:common_material prefix="xarm_" />
   <xacro:common_material prefix="xarm_gripper_" />
+  <!-- Determine which plugin to use -->
+  <xacro:property name="control_plugin" value="$(arg use_real_hardware)"/>
+  <xacro:if value="${control_plugin}">
+    <xacro:property name="ros2_control_plugin" value="uf_robot_hardware/UFRobotSystemHardware"/>
+    <xacro:property name="robot_ip" value="192.168.1.219"/>
+  </xacro:if>
+  <xacro:unless value="${control_plugin}">
+    <xacro:property name="ros2_control_plugin" value="mock_components/GenericSystem"/>
+    <xacro:property name="robot_ip" value=""/>
+  </xacro:unless>
   <!-- Instantiate the xArm6 robot with xarm prefix -->
   <xacro:xarm6_robot
@@ -31,6 +43,6 @@
     add_gripper="true"
     add_bio_gripper="false"
-    ros2_control_plugin="uf_robot_hardware/UFRobotSystemHardware"
-    robot_ip=""
+    ros2_control_plugin="${ros2_control_plugin}"
+    robot_ip="${robot_ip}"
     report_type="normal"
     baud_checkset="true"
@@ -41,5 +53,5 @@
     hard_interface="PositionJointInterface" />
   <xacro:xarm6_transmission prefix="xarm_" />
-  <xacro:xarm6_ros2_control
+  <!--<xacro:xarm6_ros2_control
     prefix="xarm_"
     hw_ns="xarm"
@@ -47,13 +59,13 @@
     add_gripper="true"
     add_bio_gripper="false"
-    ros2_control_plugin="uf_robot_hardware/UFRobotSystemHardware"
-    robot_ip="192.168.1.219"
+    ros2_control_plugin="${ros2_control_plugin}"
+    robot_ip="${robot_ip}"
     report_type="normal"
     baud_checkset="true"
-    default_gripper_baud="2000000" />
+    default_gripper_baud="2000000" /> -->
   <xacro:xarm_gripper_transmission prefix="xarm_gripper_" hard_interface="PositionJointInterface" />
-  <xacro:xarm_gripper_ros2_control
+  <!-- <xacro:xarm_gripper_ros2_control
     prefix="xarm_gripper_"
-    ros2_control_plugin="uf_robot_hardware/UFRobotSystemHardware" />
+    ros2_control_plugin="${ros2_control_plugin}"/> -->
   <!-- Mount the xArm6 on CHARMIE -->
   <joint name="xarm_mount_joint" type="fixed">

Commit message: Added optional connection to xarm to moveit launch

File: src/charmie_description/urdf/arm.xacro (robot description, xacro)
@@ -2,5 +2,5 @@
 <robot xmlns:xacro="http://www.ros.org/wiki/xacro">
   <!-- Add argument for hardware selection -->
-  <xacro:arg name="use_real_hardware" default="false"/>
+  <xacro:arg name="use_real_hardware" default="true"/>
   <!-- Set required flags used by xarm_description flags -->
   <xacro:property name="is_ros2" value="true"/>
@@ -29,5 +29,5 @@
   <xacro:if value="${control_plugin}">
     <xacro:property name="ros2_control_plugin" value="uf_robot_hardware/UFRobotSystemHardware"/>
-    <xacro:property name="robot_ip" value="192.168.1.219"/>
+    <xacro:property name="robot_ip" value="0192.168.1.219"/>
   </xacro:if>
   <xacro:unless value="${control_plugin}">
