Commit message: Changes to CHARMIE urdf so ros2_control can take into account revolute and prismatic joints

File: src/charmie_description/urdf/neck.xacro (robot description, xacro)
@@ -87,3 +87,24 @@
         </xacro:inertial_box>
     </link>
+    <ros2_control name="neck_system" type="system">
+        <hardware>
+            <plugin>mock_components/GenericSystem</plugin>
+        </hardware>
+        <joint name="neck_pan_joint">
+            <command_interface name="position">
+                <param name="min">${-pi}</param>
+                <param name="max">${pi}</param>
+            </command_interface>
+            <state_interface name="position"/>
+            <state_interface name="velocity"/>
+        </joint>
+        <joint name="neck_tilt_joint">
+            <command_interface name="position">
+                <param name="min">${-pi/3}</param>
+                <param name="max">${pi/3}</param>
+            </command_interface>
+            <state_interface name="position"/>
+            <state_interface name="velocity"/>
+        </joint>
+    </ros2_control>
 </robot>

File: src/charmie_description/urdf/torso.xacro (robot description, xacro)
@@ -69,5 +69,5 @@
     <link name="top_torso_link">
     </link>
-    <ros2_control name="charmie_system" type="system">
+    <ros2_control name="torso_system" type="system">
         <hardware>
                 <plugin>mock_components/GenericSystem</plugin>

Commit message: Commit to change branches 2

File: src/charmie_description/urdf/neck.xacro (robot description, xacro)
@@ -87,5 +87,5 @@
         </xacro:inertial_box>
     </link>
-    <ros2_control name="neck_system" type="system">
+    <!-- <ros2_control name="neck_system" type="system">
         <hardware>
             <plugin>mock_components/GenericSystem</plugin>
@@ -107,4 +107,4 @@
             <state_interface name="velocity"/>
         </joint>
-    </ros2_control>
+    </ros2_control> -->
 </robot>

File: src/charmie_description/urdf/torso.xacro (robot description, xacro)
@@ -69,5 +69,5 @@
     <link name="top_torso_link">
     </link>
-    <ros2_control name="torso_system" type="system">
+    <!-- <ros2_control name="torso_system" type="system">
         <hardware>
                 <plugin>mock_components/GenericSystem</plugin>
@@ -89,4 +89,4 @@
             <state_interface name="velocity"/>
         </joint>
-    </ros2_control>
+    </ros2_control> -->
 </robot>

File: src/charmie_moveit/charmie_moveit_config/config/charmie.ros2_control.xacro (robot description, xacro)
@@ -50,4 +50,36 @@
                 </state_interface>
             </joint>
+            <joint name="neck_pan_joint">
+                <command_interface name="position">
+                    <param name="min">${-pi}</param>
+                    <param name="max">${pi}</param>
+                </command_interface>
+                <state_interface name="position"/>
+                <state_interface name="velocity"/>
+            </joint>
+            <joint name="neck_tilt_joint">
+                <command_interface name="position">
+                    <param name="min">${-pi/3}</param>
+                    <param name="max">${pi/3}</param>
+                </command_interface>
+                <state_interface name="position"/>
+                <state_interface name="velocity"/>
+            </joint>
+            <joint name="legs_joint">
+                <command_interface name="position">
+                    <param name="min">0.0</param>
+                    <param name="max">0.14</param>
+                </command_interface>
+                <state_interface name="position"/>
+                <state_interface name="velocity"/>
+            </joint>
+            <joint name="torso_joint">
+                <command_interface name="position">
+                    <param name="min">0.0</param>
+                    <param name="max">1.22173</param>
+                </command_interface>
+                <state_interface name="position"/>
+                <state_interface name="velocity"/>
+            </joint>
         </ros2_control>
     </xacro:macro>
