Commit message: Added torso and legs joint to ros2 control

File: src/charmie_description/urdf/torso.xacro (robot description, xacro)
@@ -69,3 +69,24 @@
     <link name="top_torso_link">
     </link>
+    <ros2_control name="charmie_system" type="system">
+        <hardware>
+                <plugin>mock_components/GenericSystem</plugin>
+        </hardware>
+        <joint name="legs_joint">
+            <command_interface name="position">
+                <param name="min">0.0</param>
+                <param name="max">0.14</param>
+            </command_interface>
+            <state_interface name="position"/>
+            <state_interface name="velocity"/>
+        </joint>
+        <joint name="torso_joint">
+            <command_interface name="position">
+                <param name="min">0.0</param>
+                <param name="max">1.22173</param>
+            </command_interface>
+            <state_interface name="position"/>
+            <state_interface name="velocity"/>
+        </joint>
+    </ros2_control>
 </robot>

Commit message: Added environment flag to search_for_objects and matched torso's urdf with robot_state_publisher

File: src/charmie_description/urdf/torso.xacro (robot description, xacro)
@@ -6,4 +6,5 @@
     <xacro:property name="legs_width" value="0.19" />
     <xacro:property name="legs_height" value="0.51" />
+    <xacro:property name="legs_static_tf" value="0.105"/> <!-- to_make_obstacles_matrixes_match -->
     <xacro:property name="torso_height_from_legs" value="0.25" />
     <xacro:property name="torso_initial_angle_rads" value="0.15708" />
@@ -15,5 +16,5 @@
         <parent link="base_link"/>
         <child link="legs_link"/>
-        <origin xyz="0 0 ${base_height+legs_max_height_from_base-legs_range}" rpy="0 0 0"/>
+        <origin xyz="${-legs_static_tf} 0 ${base_height+legs_max_height_from_base-legs_range}" rpy="0 0 0"/>
         <axis xyz="0 0 1"/>
         <limit lower="0.0" upper="0.14" effort="1000.0" velocity="0.5"/>
