Commit message: Fix Hand Camera and its support position and orientation

File: src/charmie_description/urdf/real_hand_camera.xacro (robot description, xacro)
@@ -8,11 +8,9 @@
   <xacro:include filename="$(find realsense2_description)/urdf/_d405.urdf.xacro" />
   <xacro:include filename="$(find realsense2_description)/urdf/_materials.urdf.xacro" />
-  <xacro:include filename="$(find xarm_description)/urdf/common/common.link.xacro" />
-  <xacro:include filename="$(find xarm_description)/urdf/common/common.material.xacro" />
   <!-- HAND CAMERA SUPPORT -->
   <joint name="hand_camera_support_joint" type="fixed">
     <parent link="xarm_link6"/>
     <child link="hand_camera_support_link"/>
-    <origin xyz="0 0 0" rpy="0 0 0"/>
+    <origin xyz="0 0 0" rpy="0 0 ${-pi/2}"/>
   </joint>
   <link name="hand_camera_support_link">
@@ -35,5 +33,5 @@
     <parent link="hand_camera_support_link"/>
     <child link="hand_camera_link"/>
-    <origin xyz="0 0 0" rpy="0 0 0"/>
+    <origin xyz="0 0.0725 0.032" rpy="0 0 0"/>
   </joint>
   <link name="hand_camera_link">

Commit message: Understood where wrong transform is happening

File: src/charmie_description/urdf/real_hand_camera.xacro (robot description, xacro)
@@ -12,5 +12,6 @@
     <parent link="xarm_link6"/>
     <child link="hand_camera_support_link"/>
-    <origin xyz="0 0 0" rpy="0 0 ${-pi/2}"/>
+    <!-- <origin xyz="0 0 0" rpy="0 0 ${-pi/2}"/> -->
+    <origin xyz="0 0 0" rpy="0 0 0"/>
   </joint>
   <link name="hand_camera_support_link">

Commit message: Fix transform bug for hand/gripper camera

File: src/charmie_description/urdf/real_hand_camera.xacro (robot description, xacro)
@@ -12,6 +12,5 @@
     <parent link="xarm_link6"/>
     <child link="hand_camera_support_link"/>
-    <!-- <origin xyz="0 0 0" rpy="0 0 ${-pi/2}"/> -->
-    <origin xyz="0 0 0" rpy="0 0 0"/>
+    <origin xyz="0 0 0" rpy="0 0 ${-pi/2}"/>
   </joint>
   <link name="hand_camera_support_link">
@@ -34,9 +33,9 @@
     <parent link="hand_camera_support_link"/>
     <child link="hand_camera_link"/>
-    <origin xyz="0 0.0725 0.032" rpy="0 0 0"/>
+    <origin xyz="0 0.0725 0.032" rpy="${-pi/2} ${-pi/2} 0"/>
   </joint>
   <link name="hand_camera_link">
     <visual>
-      <origin xyz="0 0 0" rpy="0 0 0"/>
+      <origin xyz="0 0 0" rpy="${pi/2} 0 ${pi/2}"/>
       <geometry>
         <mesh filename="${camera_mesh_path}/d405.${mesh_suffix}" scale="0.001 0.001 0.001"/>
@@ -45,5 +44,5 @@
     </visual>
     <collision>
-      <origin xyz="0 0 0" rpy="0 0 0"/>
+      <origin xyz="0 0 0" rpy="${pi/2} 0 ${pi/2}"/>
       <geometry>
         <mesh filename="${camera_mesh_path}/d405.${mesh_suffix}" scale="0.001 0.001 0.001"/>
