Commit message: Added xarm gripper in arm.xacro

File: src/charmie_arm_ufactory/xarm_ros2/xarm_description/urdf/xarm6/xarm6_robot_macro.xacro (robot description, xacro)
@@ -6,5 +6,5 @@
     limited:=false
     velocity_control:=false
-    add_gripper:=false
+    add_gripper:=true
     add_bio_gripper:=false
     ros2_control_plugin:='uf_robot_hardware/UFRobotSystemHardware'
@@ -25,4 +25,16 @@
     <xacro:include filename="$(find xarm_description)/urdf/xarm6/xarm6.transmission.xacro" />
     <xacro:include filename="$(find xarm_description)/urdf/xarm6/xarm6.gazebo.xacro" />
+    <xacro:if value="${add_gripper}">
+      <xacro:include filename="$(find xarm_description)/urdf/gripper/xarm_gripper_macro.xacro" />
+      <xacro:property name="mesh_path" value="package://xarm_description/meshes"/>
+      <xacro:property name="mesh_suffix" value="stl"/>
+      <xacro:xarm_gripper_macro
+        prefix="${prefix}gripper_"
+        attach_to="${prefix}link6"
+        ns="${hw_ns}"
+        dof="6"
+        ros2_control_plugin="${ros2_control_plugin}"
+        hard_interface="${hard_interface}" />
+    </xacro:if>
     <xacro:if value="${limited}">
       <xacro:if value="${is_ros2}">

File: src/charmie_description/urdf/arm.xacro (robot description, xacro)
@@ -11,7 +11,9 @@
   <xacro:include filename="$(find xarm_description)/urdf/common/common.link.xacro" />
   <xacro:include filename="$(find xarm_description)/urdf/common/common.material.xacro" />
+  <!-- Include Gripper macro definition -->
+  <xacro:include filename="$(find xarm_description)/urdf/gripper/xarm_gripper_macro.xacro" />
   <!-- Instantiate the common materials with xarm prefix -->
   <xacro:common_material prefix="xarm_" />
-  <!-- Instantiate the xArm6 robot with a safe prefix -->
+  <!-- Instantiate the xArm6 robot with xarm prefix -->
   <xacro:xarm6_robot
     prefix="xarm_"
@@ -19,5 +21,5 @@
     limited="false"
     velocity_control="false"
-    add_gripper="false"
+    add_gripper="true"
     add_bio_gripper="false"
     ros2_control_plugin="uf_robot_hardware/UFRobotSystemHardware"
@@ -35,5 +37,5 @@
     <child link="xarm_link_base"/>
     <!-- Adjust this origin if needed for proper placement -->
-    <origin xyz="-0.12 0.06 -0.09" rpy="${pi/2} 0 0"/>
+    <origin xyz="-0.12 0.06 -0.09" rpy="${pi/2} ${pi} 0"/>
   </joint>
 </robot>
