Commit message: Added gripper to moveit configurated file

File: src/charmie_moveit/charmie_moveit_config/config/charmie.ros2_control.xacro (robot description, xacro)
@@ -44,4 +44,10 @@
                 </state_interface>
             </joint>
+            <joint name="xarm_gripper_drive_joint">
+                <command_interface name="position"/>
+                <state_interface name="position">
+                  <param name="initial_value">${initial_positions['xarm_gripper_drive_joint']}</param>
+                </state_interface>
+            </joint>
         </ros2_control>
     </xacro:macro>
