Commit message: Fixed xarm_gripper ros2_control error

File: src/charmie_arm_ufactory/xarm_ros2/xarm_description/urdf/gripper/xarm_gripper.ros2_control.xacro (robot description, xacro)
@@ -9,4 +9,6 @@
       <joint name="${prefix}drive_joint">
         <command_interface name="position">
+          <param name="min">0.0</param>
+          <param name="max">0.85</param>
         </command_interface>
         <command_interface name="velocity">
@@ -16,6 +18,35 @@
         <state_interface name="position"/>
         <state_interface name="velocity"/>
-        <!-- <state_interface name="effort"/> -->
       </joint>
+      <!-- <joint name="${prefix}_left_finger_joint">
+          <param name="mimic">${prefix}_drive_joint</param>
+          <param name="multiplier">1.0</param>
+          <state_interface name="position"/>
+          <state_interface name="velocity"/>
+        </joint>
+        <joint name="${prefix}_left_inner_knuckle_joint">
+          <param name="mimic">${prefix}_drive_joint</param>
+          <param name="multiplier">1.0</param>
+          <state_interface name="position"/>
+          <state_interface name="velocity"/>
+        </joint>
+        <joint name="${prefix}_right_outer_knuckle_joint">
+          <param name="mimic">${prefix}_drive_joint</param>
+          <param name="multiplier">1.0</param>
+          <state_interface name="position"/>
+          <state_interface name="velocity"/>
+        </joint>
+        <joint name="${prefix}_right_finger_joint">
+          <param name="mimic">${prefix}_drive_joint</param>
+          <param name="multiplier">1.0</param>
+          <state_interface name="position"/>
+          <state_interface name="velocity"/>
+        </joint>
+        <joint name="${prefix}_right_inner_knuckle_joint">
+          <param name="mimic">${prefix}_drive_joint</param>
+          <param name="multiplier">1.0</param>
+          <state_interface name="position"/>
+          <state_interface name="velocity"/>
+        </joint> -->
     </ros2_control>
   </xacro:macro>

File: src/charmie_arm_ufactory/xarm_ros2/xarm_description/urdf/xarm6/xarm6.ros2_control.xacro (robot description, xacro)
@@ -125,49 +125,4 @@
         <!-- <state_interface name="effort"/> -->
       </joint>
-      <xacro:if value="${add_gripper}">
-        <joint name="${prefix}gripper_drive_joint">
-          <command_interface name="position">
-            <param name="min">0</param>
-            <param name="max">0.85</param>
-          </command_interface>
-          <command_interface name="velocity">
-            <param name="min">-3.14</param>
-            <param name="max">3.14</param>
-          </command_interface>
-          <state_interface name="position"/>
-        </joint>
-        <xacro:unless value="${ros2_control_plugin == 'uf_robot_hardware/UFRobotSystemHardware'}">
-          <joint name="${prefix}gripper_left_finger_joint">
-            <param name="mimic">${prefix}gripper_drive_joint</param>
-            <param name="multiplier">1.0</param>
-            <state_interface name="position"/>
-            <state_interface name="velocity"/>
-          </joint>
-          <joint name="${prefix}gripper_left_inner_knuckle_joint">
-            <param name="mimic">${prefix}gripper_drive_joint</param>
-            <param name="multiplier">1.0</param>
-            <state_interface name="position"/>
-            <state_interface name="velocity"/>
-          </joint>
-          <joint name="${prefix}gripper_right_outer_knuckle_joint">
-            <param name="mimic">${prefix}gripper_drive_joint</param>
-            <param name="multiplier">1.0</param>
-            <state_interface name="position"/>
-            <state_interface name="velocity"/>
-          </joint>
-          <joint name="${prefix}gripper_right_finger_joint">
-            <param name="mimic">${prefix}gripper_drive_joint</param>
-            <param name="multiplier">1.0</param>
-            <state_interface name="position"/>
-            <state_interface name="velocity"/>
-          </joint>
-          <joint name="${prefix}gripper_right_inner_knuckle_joint">
-            <param name="mimic">${prefix}gripper_drive_joint</param>
-            <param name="multiplier">1.0</param>
-            <state_interface name="position"/>
-            <state_interface name="velocity"/>
-          </joint>
-        </xacro:unless>
-      </xacro:if>
     </ros2_control>
   </xacro:macro>
